Commit message: fixed leg's COG origin

File: champ_description/urdf/leg.urdf.xacro (robot description, xacro)
@@ -41,4 +41,5 @@
         <link name="${leg}_upper_leg_link">
             <inertial>
+                <origin xyz="0.065 0 0" />
                 <mass value="${upper_leg_mass}" />
                 <inertia ixx="${(1/12) * upper_leg_mass * (upper_leg_y_length * upper_leg_y_length + upper_leg_z_length * upper_leg_z_length)}" ixy="0.0" ixz="0.0"
@@ -62,4 +63,5 @@
         <link name="${leg}_lower_leg_link">
             <inertial>
+                <origin xyz="0.065 0 0" />
                 <mass value="${lower_leg_mass}" />
                 <inertia ixx="${(1/12) * lower_leg_mass * (lower_leg_y_length * lower_leg_y_length + lower_leg_z_length * lower_leg_z_length)}" ixy="0.0" ixz="0.0"

Commit message: fixed velocity,friction, and effort

File: champ_description/urdf/leg.urdf.xacro (robot description, xacro)
@@ -39,4 +39,7 @@
             </visual>
         </link>
+        <gazebo reference="${leg}_hip_link">
+            <material>Gazebo/FlatBlack</material>
+        </gazebo>
         <link name="${leg}_upper_leg_link">
             <inertial>
@@ -61,4 +64,7 @@
             </visual>
         </link>
+        <gazebo reference="${leg}_upper_leg_link">
+            <material>Gazebo/FlatBlack</material>
+        </gazebo>
         <link name="${leg}_lower_leg_link">
             <inertial>
@@ -83,8 +89,13 @@
             </visual>
         </link>
+        <gazebo reference="${leg}_lower_leg_link">
+            <mu1>10000.0</mu1>
+            <mu2>10000.0</mu2>
+            <material>Gazebo/FlatBlack</material>
+        </gazebo>
         <link name="${leg}_foot_link" />
         <joint name="${leg}_hip_joint" type="revolute">
             <axis xyz="0 1 0" />
-            <limit effort="1000.0" lower="-${pi}" upper="${pi}" velocity="0.5" />
+            <limit effort="1000.0" lower="-${pi}" upper="${pi}" velocity="3.5" />
             <parent link="base_link" />
             <child link="${leg}_hip_link" />
@@ -93,5 +104,5 @@
         <joint name="${leg}_upper_leg_joint" type="revolute">
             <axis xyz="0 0 1" />
-            <limit effort="1000.0" lower="-${pi}" upper="${pi}" velocity="0.5" />
+            <limit effort="1000.0" lower="-${pi}" upper="${pi}" velocity="3.5" />
             <parent link="${leg}_hip_link" />
             <child link="${leg}_upper_leg_link" />
@@ -100,5 +111,5 @@
         <joint name="${leg}_lower_leg_joint" type="revolute">
             <axis xyz="0 0 1" />
-            <limit effort="1000.0" lower="-${pi}" upper="${pi}" velocity="0.5" />
+            <limit effort="1000.0" lower="-${pi}" upper="${pi}" velocity="3.5" />
             <parent link="${leg}_upper_leg_link" />
             <child link="${leg}_lower_leg_link" />

Commit message: added contact parameters

File: champ_description/urdf/leg.urdf.xacro (robot description, xacro)
@@ -90,4 +90,9 @@
         </link>
         <gazebo reference="${leg}_lower_leg_link">
+            <kp>1000000.0</kp>
+            <kd>1.0</kd>
+            <mu1>0.8</mu1>
+            <mu2>0.8</mu2>
+            <maxVel>0.0</maxVel>
             <minDepth>0.001</minDepth>
             <material>Gazebo/FlatBlack</material>
@@ -96,5 +101,5 @@
         <joint name="${leg}_hip_joint" type="revolute">
             <axis xyz="0 1 0" />
-            <limit effort="1000.0" lower="-${pi}" upper="${pi}" velocity="3.5" />
+            <limit effort="20.0" lower="-${pi}" upper="${pi}" velocity="1" />
             <parent link="base_link" />
             <child link="${leg}_hip_link" />
@@ -103,5 +108,5 @@
         <joint name="${leg}_upper_leg_joint" type="revolute">
             <axis xyz="0 0 1" />
-            <limit effort="1000.0" lower="-${pi}" upper="${pi}" velocity="3.5" />
+            <limit effort="20.0" lower="-${pi}" upper="${pi}" velocity="3.5" />
             <parent link="${leg}_hip_link" />
             <child link="${leg}_upper_leg_link" />
@@ -110,5 +115,5 @@
         <joint name="${leg}_lower_leg_joint" type="revolute">
             <axis xyz="0 0 1" />
-            <limit effort="1000.0" lower="-${pi}" upper="${pi}" velocity="3.5" />
+            <limit effort="20.0" lower="-${pi}" upper="${pi}" velocity="3.5" />
             <parent link="${leg}_upper_leg_link" />
             <child link="${leg}_lower_leg_link" />

Commit message: fine tuned effort and velocity for leg joints for lesser jerks

File: champ_description/urdf/leg.urdf.xacro (robot description, xacro)
@@ -101,5 +101,5 @@
         <joint name="${leg}_hip_joint" type="revolute">
             <axis xyz="0 1 0" />
-            <limit effort="20.0" lower="-${pi}" upper="${pi}" velocity="1" />
+            <limit effort="50" lower="-${pi}" upper="${pi}" velocity="2.0" />
             <parent link="base_link" />
             <child link="${leg}_hip_link" />
@@ -108,5 +108,5 @@
         <joint name="${leg}_upper_leg_joint" type="revolute">
             <axis xyz="0 0 1" />
-            <limit effort="20.0" lower="-${pi}" upper="${pi}" velocity="3.5" />
+            <limit effort="50" lower="-${pi}" upper="${pi}" velocity="2.0" />
             <parent link="${leg}_hip_link" />
             <child link="${leg}_upper_leg_link" />
@@ -115,5 +115,5 @@
         <joint name="${leg}_lower_leg_joint" type="revolute">
             <axis xyz="0 0 1" />
-            <limit effort="20.0" lower="-${pi}" upper="${pi}" velocity="3.5" />
+            <limit effort="50" lower="-${pi}" upper="${pi}" velocity="2.0" />
             <parent link="${leg}_upper_leg_link" />
             <child link="${leg}_lower_leg_link" />

File: champ_description/urdf/properties.urdf.xacro (robot description, xacro)
@@ -22,5 +22,5 @@
     <xacro:property name="lower_leg_z_length" value="0.022" />
     <xacro:property name="base_mesh_path" value="package://champ_description/meshes/base.stl" />
-    <xacro:property name="base_mass" value="5.0" />
+    <xacro:property name="base_mass" value="3.0" />
     <xacro:property name="base_x_length" value="0.5" />
     <xacro:property name="base_y_length" value="0.29" />

Commit message: fine tuned for smoother walking

File: champ_description/urdf/leg.urdf.xacro (robot description, xacro)
@@ -101,5 +101,5 @@
         <joint name="${leg}_hip_joint" type="revolute">
             <axis xyz="0 1 0" />
-            <limit effort="50" lower="-${pi}" upper="${pi}" velocity="2.0" />
+            <limit effort="20" lower="-${pi}" upper="${pi}" velocity="2.0" />
             <parent link="base_link" />
             <child link="${leg}_hip_link" />
@@ -108,5 +108,5 @@
         <joint name="${leg}_upper_leg_joint" type="revolute">
             <axis xyz="0 0 1" />
-            <limit effort="50" lower="-${pi}" upper="${pi}" velocity="2.0" />
+            <limit effort="20" lower="-${pi}" upper="${pi}" velocity="2.0" />
             <parent link="${leg}_hip_link" />
             <child link="${leg}_upper_leg_link" />
@@ -115,5 +115,5 @@
         <joint name="${leg}_lower_leg_joint" type="revolute">
             <axis xyz="0 0 1" />
-            <limit effort="50" lower="-${pi}" upper="${pi}" velocity="2.0" />
+            <limit effort="20" lower="-${pi}" upper="${pi}" velocity="2.0" />
             <parent link="${leg}_upper_leg_link" />
             <child link="${leg}_lower_leg_link" />

Commit message: match new model orientation

File: champ_description/urdf/leg.urdf.xacro (robot description, xacro)
@@ -103,31 +103,32 @@
             <parent link="base_link" />
             <child link="${leg}_hip_debug_link" />
-            <origin xyz="${base_to_hip_xyz}" rpy="0 ${pi/2} ${pi/2}" />
+            <origin xyz="${base_to_hip_xyz}" rpy="0 0 0" />
         </joint>
         <joint name="${leg}_hip_joint" type="revolute">
-            <axis xyz="0 1 0" />
+            <axis xyz="1 0 0" />
             <limit effort="25" lower="-${pi}" upper="${pi}" velocity="1.5" />
             <parent link="base_link" />
             <child link="${leg}_hip_link" />
-            <origin xyz="${base_to_hip_xyz}" rpy="-${pi/2} ${pi/2} 0" />
+            <origin xyz="${base_to_hip_xyz}" rpy="0 0 0" />
         </joint>
         <joint name="${leg}_upper_leg_joint" type="revolute">
-            <axis xyz="0 0 1" />
+            <axis xyz="0 1 0" />
             <limit effort="25" lower="-${pi}" upper="${pi}" velocity="1.5" />
             <parent link="${leg}_hip_link" />
             <child link="${leg}_upper_leg_link" />
-            <origin xyz="0 0 ${hip_to_upper_leg}" rpy="0 0 0" />
+            <origin xyz="0 ${hip_to_upper_leg} 0" rpy="0 0 0" />
         </joint>
         <joint name="${leg}_lower_leg_joint" type="revolute">
-            <axis xyz="0 0 1" />
+            <axis xyz="0 1 0" />
             <limit effort="25" lower="-${pi}" upper="${pi}" velocity="1.5" />
             <parent link="${leg}_upper_leg_link" />
             <child link="${leg}_lower_leg_link" />
-            <origin xyz="${upper_leg_to_lower_leg_distance} 0 0" rpy="0 0 0" />
+            <origin xyz="0 0 -${upper_leg_to_lower_leg_distance}" rpy="0 0 0" />
         </joint>
         <joint name="${leg}_foot_joint" type="fixed">
             <parent link="${leg}_lower_leg_link" />
             <child link="${leg}_foot_link" />
-            <origin xyz="${lower_leg_to_foot_distance} 0 0" rpy="0 0 0" />
+            <!-- <origin xyz="0.00325 0 -${lower_leg_to_foot_distance}" rpy="0 0 0" /> -->
+            <origin xyz="0 0 -${lower_leg_to_foot_distance}" rpy="0 0 0" />
         </joint>
         <transmission name="${leg}_hip_joint_trans">

Commit message: fixed code to match newly reorientated frames

File: champ_description/urdf/leg.urdf.xacro (robot description, xacro)
@@ -45,5 +45,5 @@
         <link name="${leg}_upper_leg_link">
             <inertial>
-                <origin xyz="${(upper_leg_x_length / 2) - ((upper_leg_x_length - upper_leg_to_lower_leg_distance) / 2)} 0 0" />
+                <origin xyz="0 0 -${(upper_leg_z_length / 2) - ((upper_leg_z_length - upper_leg_to_lower_leg_distance) / 2)}" />
                 <mass value="${upper_leg_mass}" />
                 <inertia ixx="${(1/12) * upper_leg_mass * (upper_leg_y_length * upper_leg_y_length + upper_leg_z_length * upper_leg_z_length)}" ixy="0.0" ixz="0.0"
@@ -70,5 +70,5 @@
         <link name="${leg}_lower_leg_link">
             <inertial>
-                <origin xyz="${(lower_leg_to_foot_distance - (lower_leg_x_length - lower_leg_to_foot_distance)) / 2} 0 0" />
+                <origin xyz="0 0 -${(lower_leg_to_foot_distance - (lower_leg_z_length - lower_leg_to_foot_distance)) / 2}" />
                 <mass value="${lower_leg_mass}" />
                 <inertia ixx="${(1/12) * lower_leg_mass * (lower_leg_y_length * lower_leg_y_length + lower_leg_z_length * lower_leg_z_length)}" ixy="0.0" ixz="0.0"

File: champ_description/urdf/properties.urdf.xacro (robot description, xacro)
@@ -8,17 +8,17 @@
     <xacro:property name="hip_mesh_path" value="package://champ_description/meshes/hip.stl" />
     <xacro:property name="hip_mass" value="0.250" />
-    <xacro:property name="hip_x_length" value="0.130" />
-    <xacro:property name="hip_y_length" value="0.112" />
-    <xacro:property name="hip_z_length" value="0.08" />
+    <xacro:property name="hip_x_length" value="0.112" />
+    <xacro:property name="hip_y_length" value="0.08" />
+    <xacro:property name="hip_z_length" value="0.130" />
     <xacro:property name="upper_leg_mesh_path" value="package://champ_description/meshes/upper_leg.stl" />
     <xacro:property name="upper_leg_mass" value="0.125" />
-    <xacro:property name="upper_leg_x_length" value="0.1905" />
-    <xacro:property name="upper_leg_y_length" value="0.05" />
-    <xacro:property name="upper_leg_z_length" value="0.03" />
+    <xacro:property name="upper_leg_x_length" value="0.05" />
+    <xacro:property name="upper_leg_y_length" value="0.03" />
+    <xacro:property name="upper_leg_z_length" value="0.1905" />
     <xacro:property name="lower_leg_mesh_path" value="package://champ_description/meshes/lower_leg.stl" />
     <xacro:property name="lower_leg_mass" value="0.125" />
-    <xacro:property name="lower_leg_x_length" value="0.156" />
-    <xacro:property name="lower_leg_y_length" value="0.039" />
-    <xacro:property name="lower_leg_z_length" value="0.022" />
+    <xacro:property name="lower_leg_x_length" value="0.039" />
+    <xacro:property name="lower_leg_y_length" value="0.022" />
+    <xacro:property name="lower_leg_z_length" value="0.156" />
     <xacro:property name="base_mesh_path" value="package://champ_description/meshes/base.stl" />
     <xacro:property name="base_mass" value="3.0" />
