Commit message: split simulated sensors into a separate xacro

File: champ_description/urdf/champ.urdf (robot description, URDF)
Before this commit: robot champ, 30 links, 29 joints
Links:
- removed link camera_base_frame
- removed link camera_depth_frame
- removed link camera_depth_optical_frame
- removed link camera_link
- removed link camera_rgb_frame
- removed link camera_rgb_optical_frame
- removed link hokuyo_frame
- removed link hokuyo_scan_link
- removed link imu_link
Joints:
- removed joint camera_base_joint
- removed joint camera_depth_joint
- removed joint camera_depth_optical_joint
- removed joint camera_joint
- removed joint camera_rgb_joint
- removed joint camera_rgb_optical_joint
- removed joint hokuyo_joint
- removed joint hokuyo_scan_joint
- removed joint imu_joint

File: champ_description/urdf/champ.urdf.xacro (robot description, xacro)
@@ -33,57 +33,12 @@
         <material>Gazebo/FlatBlack</material>
     </gazebo>
-    <link name="imu_link">
-        <inertial>
-            <mass value="0.001"/>
-            <origin xyz="0 0 0" rpy="0 0 0"/>
-            <inertia ixx="1e-09" ixy="0.0" ixz="0.0" iyy="1e-09" iyz="0.0" izz="1e-09"/>
-        </inertial>
-    </link>
-    <joint name="imu_joint" type="fixed">
-        <parent link="base_link" />
-        <child link="imu_link" />
-    </joint>
     <xacro:include filename="$(find champ_description)/urdf/leg.urdf.xacro" />
+    <xacro:if value="$(optenv ENABLE_SENSORS 0)">
+        <xacro:include filename="$(find champ_description)/urdf/accessories.urdf.xacro" />
+    </xacro:if>
     <xacro:champ_leg leg="lf"/>
     <xacro:champ_leg leg="lh"/>
     <xacro:champ_leg leg="rf"/>
     <xacro:champ_leg leg="rh"/>
-    <xacro:include filename="$(find common_sensors)/urdf/sensors/hokuyo_utm30lx.urdf.xacro" />
-    <xacro:hokuyo_utm30lx
-        name="hokuyo"
-        parent="base_link"
-        ros_topic="scan"
-        update_rate="30"
-        ray_count="1040"
-        min_angle="130"
-        max_angle="-130" >
-        <origin xyz="0.0 0.0 ${base_z_length / 2 + 0.04}" rpy="0 0 0"/>
-    </xacro:hokuyo_utm30lx>
-    <gazebo reference="hokuyo_frame">
-		<material>Gazebo/FlatBlack</material>
-	</gazebo>
-    <xacro:include filename="$(find common_sensors)/urdf/sensors/xtion.urdf.xacro" />
-    <xacro:sensor_xtion
-        parent="base_link"
-        camera_name="camera">
-        <origin xyz="${base_x_length / 2} 0.0 ${base_z_length / 2 + 0.01}" rpy="0 0 0"/>
-    </xacro:sensor_xtion>
-    <gazebo reference="hokuyo_frame">
-		<material>Gazebo/FlatBlack</material>
-	</gazebo>
-    <gazebo>
-        <plugin name="imu_controller" filename="libhector_gazebo_ros_imu.so">
-            <robotNamespace>/</robotNamespace>
-            <updateRate>50.0</updateRate>
-            <bodyName>imu_link</bodyName>
-            <topicName>imu/data</topicName>
-            <accelDrift>0.005 0.005 0.005</accelDrift>
-            <accelGaussianNoise>0.005 0.005 0.005</accelGaussianNoise>
-            <rateDrift>0.005 0.005 0.005 </rateDrift>
-            <rateGaussianNoise>0.005 0.005 0.005 </rateGaussianNoise>
-            <headingDrift>0.005</headingDrift>
-            <headingGaussianNoise>0.005</headingGaussianNoise>
-        </plugin>
-    </gazebo>
     <gazebo>
       <plugin name="p3d_base_controller" filename="libgazebo_ros_p3d.so">

Commit message: regenerated to update changes

File: champ_description/urdf/champ.urdf (robot description, URDF)
Before this commit: robot champ, 28 links, 27 joints
Links:
- link base_link: mass 3.0 -> 2.0

Commit message: changed default urdf to have sensors attached

File: champ_description/urdf/champ.urdf (robot description, URDF)
Before this commit: robot champ, 21 links, 20 joints
Links:
- added link camera_depth_frame
- added link camera_depth_optical_frame
- added link camera_link, mass 0.200; collision mesh filename=package://hector_sensors_description/meshes/asus_camera/asu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; visual mesh filename=package://hector_sensors_description/meshes/asus_camera/asu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
- added link camera_rgb_frame
- added link camera_rgb_optical_frame
- added link hokuyo_frame, mass 0.270; collision box size=0.058 0.058 0.087; visual mesh filename=package://hector_sensors_description/meshes/hokuyo_utm30lx/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
- added link imu_link, mass 0.001
Joints:
- added joint camera_depth_joint: type fixed, parent camera_link, child camera_depth_frame, origin xyz=0.0 0.049 0.0 rpy=0 0 0
- added joint camera_depth_optical_joint: type fixed, parent camera_depth_frame, child camera_depth_optical_frame, origin xyz=0 0 0 rpy=-1.57079632679 0.0 -1.57079632679
- added joint camera_joint: type fixed, parent base_link, child camera_link, origin xyz=0.25 0.0 0.075 rpy=0 0 0
- added joint camera_rgb_joint: type fixed, parent camera_link, child camera_rgb_frame, origin xyz=0.0 0.022 0.0 rpy=0 0 0
- added joint camera_rgb_optical_joint: type fixed, parent camera_rgb_frame, child camera_rgb_optical_frame, origin xyz=0 0 0 rpy=-1.57079632679 0.0 -1.57079632679
- added joint hokuyo_joint: type fixed, parent base_link, child hokuyo_frame, origin xyz=0.0 0.0 0.105 rpy=0 0 0
- added joint imu_joint: type fixed, parent base_link, child imu_link

Commit message: separated inertia from base_link to a dummy link

File: champ_description/urdf/champ.urdf (robot description, URDF)
Before this commit: robot champ, 28 links, 27 joints
Links:
- added link base_inertia, mass 2.0
- link base_link: mass 2.0 -> None
Joints:
- added joint base_link_to_base_inertia: type fixed, parent base_link, child base_inertia, origin xyz=0 0 0 rpy=0 0 0

File: champ_description/urdf/champ.urdf.xacro (robot description, xacro)
@@ -3,13 +3,5 @@
     <xacro:include filename="$(find champ_description)/urdf/properties.urdf.xacro" />
     <material name="black"><color rgba="0.15 0.15 0.15 1.0" /></material>
-    <!-- <link name="champ"/> -->
     <link name="base_link">
-        <inertial>
-            <origin xyz="0 0 0" />
-            <mass value="${base_mass}" />
-            <inertia ixx="${(1/12) * base_mass * (base_y_length * base_y_length + base_z_length * base_z_length)}" ixy="0.0" ixz="0.0"
-                     iyy="${(1/12) * base_mass * (base_x_length * base_x_length + base_z_length * base_z_length)}" iyz="0.0"
-                     izz="${(1/12) * base_mass * (base_x_length * base_x_length + base_y_length * base_y_length)}" />
-        </inertial>
         <collision>
             <origin xyz="0 0 0" rpy="0 0 0" />
@@ -26,4 +18,18 @@
         </visual>
     </link>
+    <link name="base_inertia">
+        <inertial>
+            <origin xyz="0 0 0" />
+            <mass value="${base_mass}" />
+            <inertia ixx="${(1/12) * base_mass * (base_y_length * base_y_length + base_z_length * base_z_length)}" ixy="0.0" ixz="0.0"
+                     iyy="${(1/12) * base_mass * (base_x_length * base_x_length + base_z_length * base_z_length)}" iyz="0.0"
+                     izz="${(1/12) * base_mass * (base_x_length * base_x_length + base_y_length * base_y_length)}" />
+        </inertial>
+    </link>
+    <joint name="base_link_to_base_inertia" type="fixed">
+        <parent link="base_link"/>
+        <child link="base_inertia"/>
+        <origin rpy="0 0 0" xyz="0 0 0"/>
+    </joint>
     <gazebo reference="base_link">
         <material>Gazebo/FlatBlack</material>
