Commit message: added debug link

File: champ_description/urdf/champ_arm.urdf (robot description, URDF)
Before this commit: robot champ, 29 links, 28 joints
Links:
- added link upper_arm_debug_link
Joints:
- added joint upper_arm_debug_joint: type fixed, parent base, child upper_arm_debug_link, origin xyz=0 0 0.035 rpy=0 0 0

Commit message: fixed missing arm meshes

File: champ_description/urdf/champ_arm.urdf (robot description, URDF)
Before this commit: robot champ, 30 links, 29 joints
Links:
- link base: geometry collision mesh filename=package://champ_description/meshes/arm/base.stl scale=0.001 0.001 0.001; visual mesh filename=package://champ_description/meshes/arm/base.stl scale=0.001 0.001 0.001
- link lower_arm: geometry collision mesh filename=package://champ_description/meshes/arm/lower_arm.stl scale=0.001 0.001 0.001; visual mesh filename=package://champ_description/meshes/arm/lower_arm.stl scale=0.001 0.001 0.001
- link upper_arm: geometry collision mesh filename=package://champ_description/meshes/arm/upper_arm.stl scale=0.001 0.001 0.001; visual mesh filename=package://champ_description/meshes/arm/upper_arm.stl scale=0.001 0.001 0.001
- link wrist1: geometry collision mesh filename=package://champ_description/meshes/arm/wrist1.stl scale=0.001 0.001 0.001; visual mesh filename=package://champ_description/meshes/arm/wrist1.stl scale=0.001 0.001 0.001
- link wrist2: geometry collision mesh filename=package://champ_description/meshes/arm/wrist2.stl scale=0.001 0.001 0.001; visual mesh filename=package://champ_description/meshes/arm/wrist2.stl scale=0.001 0.001 0.001
