Commit message: working ik test

File: champ_description/urdf/champ.urdf.xacro (robot description, xacro)
@@ -27,4 +27,10 @@
         <origin xyz="0 0 0" rpy="0 0 0" />
     </joint>
+        <link name="hip_debug_link"/>
+    <joint name="base_to_debug_link" type="fixed">
+        <parent link="base_link" />
+        <child link="hip_debug_link" />
+        <origin xyz="0.1675 0.105 0" rpy="0 1.5708 -1.5708" />
+    </joint>
     <xacro:include filename="$(find champ_description)/urdf/leg.urdf.xacro" />
     <xacro:champ_leg leg="lf"/>

Commit message: flipped right legs to match hip ik

File: champ_description/urdf/champ.urdf.xacro (robot description, xacro)
@@ -3,5 +3,5 @@
     <xacro:property name="base_to_hip_x" value="0.1675" />
     <xacro:property name="base_to_hip_y" value="0.105" />
-    <xacro:property name="hip_to_upper_leg_distance" value="-0.071" />
+    <xacro:property name="hip_to_upper_leg_distance" value="0.071" />
     <xacro:property name="upper_leg_to_lower_leg_distance" value="0.141" />
     <xacro:property name="lower_leg_to_ee_distance" value="0.141" />
@@ -31,5 +31,5 @@
         <parent link="base_link" />
         <child link="hip_debug_link" />
-        <origin xyz="0.1675 0.105 0" rpy="0 1.5708 -1.5708" />
+        <origin xyz="0.1675 -0.105 0" rpy="0 1.5708 -1.5708" />
     </joint>
     <xacro:include filename="$(find champ_description)/urdf/leg.urdf.xacro" />

File: champ_description/urdf/leg.urdf.xacro (robot description, xacro)
@@ -5,20 +5,23 @@
             <xacro:property name="base_to_hip_xyz" value="${base_to_hip_x} ${base_to_hip_y} 0" />
             <!-- <xacro:property name="base_to_hip_rpy" value="${pi/2} ${pi/2} 0" /> -->
-            <xacro:property name="base_to_hip_rpy" value="${pi/2} ${pi/2} 0" />
+            <xacro:property name="hip_to_upper_leg" value="-${hip_to_upper_leg_distance}" />
             <xacro:property name="lower_leg_rpy" value="0 0 0" />
         </xacro:if>
         <xacro:if value="${leg == 'rf'}">
             <xacro:property name="base_to_hip_xyz" value="${base_to_hip_x} -${base_to_hip_y} 0" />
-            <xacro:property name="base_to_hip_rpy" value="-${pi/2} ${pi/2} 0" />
+            <!-- <xacro:property name="base_to_hip_rpy" value="${pi/2} ${pi/2} 0" /> -->
+            <xacro:property name="hip_to_upper_leg" value="${hip_to_upper_leg_distance}" />
             <xacro:property name="lower_leg_rpy" value="${pi} 0 0" />
         </xacro:if>
         <xacro:if value="${leg == 'lr'}">
             <xacro:property name="base_to_hip_xyz" value="-${base_to_hip_x} ${base_to_hip_y} 0" />
-            <xacro:property name="base_to_hip_rpy" value="${pi/2} ${pi/2} 0" />
+            <!-- <xacro:property name="base_to_hip_rpy" value="${pi/2} ${pi/2} 0" /> -->
+            <xacro:property name="hip_to_upper_leg" value="-${hip_to_upper_leg_distance}" />
             <xacro:property name="lower_leg_rpy" value="0 0 0" />
         </xacro:if>
         <xacro:if value="${leg == 'rr'}">
             <xacro:property name="base_to_hip_xyz" value="-${base_to_hip_x} -${base_to_hip_y} 0" />
-            <xacro:property name="base_to_hip_rpy" value="-${pi/2} ${pi/2} 0" />
+            <!-- <xacro:property name="base_to_hip_rpy" value="${pi/2} ${pi/2} 0" /> -->
+            <xacro:property name="hip_to_upper_leg" value="${hip_to_upper_leg_distance}" />
             <xacro:property name="lower_leg_rpy" value="${pi} 0 0" />
         </xacro:if>
@@ -37,5 +40,5 @@
             <parent link="base_link" />
             <child link="${leg}_hip_link" />
-            <origin xyz="${base_to_hip_xyz}" rpy="${base_to_hip_rpy}" />
+            <origin xyz="${base_to_hip_xyz}" rpy="${pi/2} ${pi/2} 0" />
         </joint>
         <link name="${leg}_upper_leg_link">
@@ -53,5 +56,5 @@
             <parent link="${leg}_hip_link" />
             <child link="${leg}_upper_leg_link" />
-            <origin xyz="0 0 ${hip_to_upper_leg_distance}" rpy="0 0 0" />
+            <origin xyz="0 0 ${hip_to_upper_leg}" rpy="0 0 0" />
         </joint>
         <link name="${leg}_lower_leg_link">

Commit message: rotated legs + pi/2

File: champ_description/urdf/champ.urdf.xacro (robot description, xacro)
@@ -27,10 +27,16 @@
         <origin xyz="0 0 0" rpy="0 0 0" />
     </joint>
-        <link name="hip_debug_link"/>
+    <link name="lf_hip_debug_link"/>
     <joint name="base_to_debug_link" type="fixed">
         <parent link="base_link" />
-        <child link="hip_debug_link" />
-        <origin xyz="0.1675 -0.105 0" rpy="0 1.5708 -1.5708" />
+        <child link="lf_hip_debug_link" />
+        <origin xyz="0.1675 0.105 0" rpy="0 ${pi/2} ${pi/2}" />
     </joint>
+    <!-- <link name="rf_hip_debug_link"/>
+    <joint name="base_to_debug_link" type="fixed">
+        <parent link="base_link" />
+        <child link="rf_hip_debug_link" />
+        <origin xyz="0.1675 -0.105 0" rpy="0 ${pi/2} ${pi/2}" />
+    </joint> -->
     <xacro:include filename="$(find champ_description)/urdf/leg.urdf.xacro" />
     <xacro:champ_leg leg="lf"/>

File: champ_description/urdf/leg.urdf.xacro (robot description, xacro)
@@ -4,24 +4,20 @@
         <xacro:if value="${leg == 'lf'}">
             <xacro:property name="base_to_hip_xyz" value="${base_to_hip_x} ${base_to_hip_y} 0" />
-            <!-- <xacro:property name="base_to_hip_rpy" value="${pi/2} ${pi/2} 0" /> -->
-            <xacro:property name="hip_to_upper_leg" value="-${hip_to_upper_leg_distance}" />
+            <xacro:property name="hip_to_upper_leg" value="${hip_to_upper_leg_distance}" />
             <xacro:property name="lower_leg_rpy" value="0 0 0" />
         </xacro:if>
         <xacro:if value="${leg == 'rf'}">
             <xacro:property name="base_to_hip_xyz" value="${base_to_hip_x} -${base_to_hip_y} 0" />
-            <!-- <xacro:property name="base_to_hip_rpy" value="${pi/2} ${pi/2} 0" /> -->
-            <xacro:property name="hip_to_upper_leg" value="${hip_to_upper_leg_distance}" />
+            <xacro:property name="hip_to_upper_leg" value="-${hip_to_upper_leg_distance}" />
             <xacro:property name="lower_leg_rpy" value="${pi} 0 0" />
         </xacro:if>
         <xacro:if value="${leg == 'lr'}">
             <xacro:property name="base_to_hip_xyz" value="-${base_to_hip_x} ${base_to_hip_y} 0" />
-            <!-- <xacro:property name="base_to_hip_rpy" value="${pi/2} ${pi/2} 0" /> -->
-            <xacro:property name="hip_to_upper_leg" value="-${hip_to_upper_leg_distance}" />
+            <xacro:property name="hip_to_upper_leg" value="${hip_to_upper_leg_distance}" />
             <xacro:property name="lower_leg_rpy" value="0 0 0" />
         </xacro:if>
         <xacro:if value="${leg == 'rr'}">
             <xacro:property name="base_to_hip_xyz" value="-${base_to_hip_x} -${base_to_hip_y} 0" />
-            <!-- <xacro:property name="base_to_hip_rpy" value="${pi/2} ${pi/2} 0" /> -->
-            <xacro:property name="hip_to_upper_leg" value="${hip_to_upper_leg_distance}" />
+            <xacro:property name="hip_to_upper_leg" value="-${hip_to_upper_leg_distance}" />
             <xacro:property name="lower_leg_rpy" value="${pi} 0 0" />
         </xacro:if>
@@ -40,5 +36,5 @@
             <parent link="base_link" />
             <child link="${leg}_hip_link" />
-            <origin xyz="${base_to_hip_xyz}" rpy="${pi/2} ${pi/2} 0" />
+            <origin xyz="${base_to_hip_xyz}" rpy="-${pi/2} ${pi/2} 0" />
         </joint>
         <link name="${leg}_upper_leg_link">

Commit message: renamed all rear legs' suffix from r to h

File: champ_description/urdf/champ.urdf.xacro (robot description, xacro)
@@ -27,20 +27,20 @@
         <origin xyz="0 0 0" rpy="0 0 0" />
     </joint>
-    <link name="lf_hip_debug_link"/>
+    <!-- <link name="lf_hip_debug_link"/>
     <joint name="base_to_debug_link" type="fixed">
         <parent link="base_link" />
         <child link="lf_hip_debug_link" />
         <origin xyz="0.1675 0.105 0" rpy="0 ${pi/2} ${pi/2}" />
-    </joint>
-    <!-- <link name="rf_hip_debug_link"/>
+    </joint> -->
+    <link name="rf_hip_debug_link"/>
     <joint name="base_to_debug_link" type="fixed">
         <parent link="base_link" />
         <child link="rf_hip_debug_link" />
         <origin xyz="0.1675 -0.105 0" rpy="0 ${pi/2} ${pi/2}" />
-    </joint> -->
+    </joint>
     <xacro:include filename="$(find champ_description)/urdf/leg.urdf.xacro" />
     <xacro:champ_leg leg="lf"/>
-    <xacro:champ_leg leg="lr"/>
+    <xacro:champ_leg leg="lh"/>
     <xacro:champ_leg leg="rf"/>
-    <xacro:champ_leg leg="rr"/>
+    <xacro:champ_leg leg="rh"/>
 </robot>

File: champ_description/urdf/leg.urdf.xacro (robot description, xacro)
@@ -5,20 +5,16 @@
             <xacro:property name="base_to_hip_xyz" value="${base_to_hip_x} ${base_to_hip_y} 0" />
             <xacro:property name="hip_to_upper_leg" value="${hip_to_upper_leg_distance}" />
-            <xacro:property name="lower_leg_rpy" value="0 0 0" />
+        </xacro:if>
+        <xacro:if value="${leg == 'lh'}">
+            <xacro:property name="base_to_hip_xyz" value="-${base_to_hip_x} ${base_to_hip_y} 0" />
+            <xacro:property name="hip_to_upper_leg" value="${hip_to_upper_leg_distance}" />
         </xacro:if>
         <xacro:if value="${leg == 'rf'}">
             <xacro:property name="base_to_hip_xyz" value="${base_to_hip_x} -${base_to_hip_y} 0" />
             <xacro:property name="hip_to_upper_leg" value="-${hip_to_upper_leg_distance}" />
-            <xacro:property name="lower_leg_rpy" value="${pi} 0 0" />
         </xacro:if>
-        <xacro:if value="${leg == 'lr'}">
-            <xacro:property name="base_to_hip_xyz" value="-${base_to_hip_x} ${base_to_hip_y} 0" />
-            <xacro:property name="hip_to_upper_leg" value="${hip_to_upper_leg_distance}" />
-            <xacro:property name="lower_leg_rpy" value="0 0 0" />
-        </xacro:if>
-        <xacro:if value="${leg == 'rr'}">
+        <xacro:if value="${leg == 'rh'}">
             <xacro:property name="base_to_hip_xyz" value="-${base_to_hip_x} -${base_to_hip_y} 0" />
             <xacro:property name="hip_to_upper_leg" value="-${hip_to_upper_leg_distance}" />
-            <xacro:property name="lower_leg_rpy" value="${pi} 0 0" />
         </xacro:if>
         <link name="${leg}_hip_link">
@@ -56,5 +52,5 @@
         <link name="${leg}_lower_leg_link">
             <visual>
-                <origin xyz="0 0 0" rpy="${lower_leg_rpy}" />
+                <origin xyz="0 0 0" rpy="0 0 0" />
                 <geometry>
                     <mesh filename="${lower_leg_mesh_path}" scale="0.001 0.001 0.001" />

Commit message: renamed each foot from ee to foot

File: champ_description/urdf/champ.urdf.xacro (robot description, xacro)
@@ -5,5 +5,5 @@
     <xacro:property name="hip_to_upper_leg_distance" value="0.071" />
     <xacro:property name="upper_leg_to_lower_leg_distance" value="0.141" />
-    <xacro:property name="lower_leg_to_ee_distance" value="0.141" />
+    <xacro:property name="lower_leg_to_foot_distance" value="0.141" />
     <xacro:property name="hip_mesh_path" value="package://champ_description/meshes/hip.stl" />
     <xacro:property name="upper_leg_mesh_path" value="package://champ_description/meshes/upper_leg.stl" />

File: champ_description/urdf/leg.urdf.xacro (robot description, xacro)
@@ -66,9 +66,9 @@
             <origin xyz="${upper_leg_to_lower_leg_distance} 0 0" rpy="0 0 0" />
         </joint>
-        <link name="${leg}_ee_link" />
-        <joint name="${leg}_ee_joint" type="fixed">
+        <link name="${leg}_foot_link" />
+        <joint name="${leg}_foot_joint" type="fixed">
             <parent link="${leg}_lower_leg_link" />
-            <child link="${leg}_ee_link" />
-            <origin xyz="${lower_leg_to_ee_distance} 0 0" rpy="0 0 0" />
+            <child link="${leg}_foot_link" />
+            <origin xyz="${lower_leg_to_foot_distance} 0 0" rpy="0 0 0" />
         </joint>
     </xacro:macro>

Commit message: added hip debug frames for displaying points all legs

File: champ_description/urdf/champ.urdf.xacro (robot description, xacro)
@@ -1,7 +1,7 @@
 <?xml version="1.0"?>
 <robot name="champ" xmlns:xacro="http://www.ros.org/wiki/xacro">
-    <xacro:property name="base_to_hip_x" value="0.1675" />
+    <xacro:property name="base_to_hip_x" value="0.175" />
     <xacro:property name="base_to_hip_y" value="0.105" />
-    <xacro:property name="hip_to_upper_leg_distance" value="0.071" />
+    <xacro:property name="hip_to_upper_leg_distance" value="0.06" />
     <xacro:property name="upper_leg_to_lower_leg_distance" value="0.141" />
     <xacro:property name="lower_leg_to_foot_distance" value="0.141" />
@@ -27,15 +27,27 @@
         <origin xyz="0 0 0" rpy="0 0 0" />
     </joint>
-    <!-- <link name="lf_hip_debug_link"/>
-    <joint name="base_to_debug_link" type="fixed">
+    <link name="lf_hip_debug_link"/>
+    <joint name="lf_debug_joint" type="fixed">
         <parent link="base_link" />
         <child link="lf_hip_debug_link" />
-        <origin xyz="0.1675 0.105 0" rpy="0 ${pi/2} ${pi/2}" />
-    </joint> -->
+        <origin xyz="${base_to_hip_x} ${base_to_hip_y} 0" rpy="0 ${pi/2} ${pi/2}" />
+    </joint>
     <link name="rf_hip_debug_link"/>
-    <joint name="base_to_debug_link" type="fixed">
+    <joint name="rf_debug_joint" type="fixed">
         <parent link="base_link" />
         <child link="rf_hip_debug_link" />
-        <origin xyz="0.1675 -0.105 0" rpy="0 ${pi/2} ${pi/2}" />
+        <origin xyz="${base_to_hip_x} -${base_to_hip_y} 0" rpy="0 ${pi/2} ${pi/2}" />
+    </joint>
+    <link name="lh_hip_debug_link"/>
+    <joint name="lh_debug_joint" type="fixed">
+        <parent link="base_link" />
+        <child link="lh_hip_debug_link" />
+        <origin xyz="-${base_to_hip_x} ${base_to_hip_y} 0" rpy="0 ${pi/2} ${pi/2}" />
+    </joint>
+    <link name="rh_hip_debug_link"/>
+    <joint name="rh_debug_joint" type="fixed">
+        <parent link="base_link" />
+        <child link="rh_hip_debug_link" />
+        <origin xyz="-${base_to_hip_x} -${base_to_hip_y} 0" rpy="0 ${pi/2} ${pi/2}" />
     </joint>
     <xacro:include filename="$(find champ_description)/urdf/leg.urdf.xacro" />
