Commit message: added gazebo sim environment

File: champ_description/urdf/champ.urdf.xacro (robot description, xacro)
@@ -1,17 +1,20 @@
 <?xml version="1.0"?>
 <robot name="champ" xmlns:xacro="http://www.ros.org/wiki/xacro">
-    <xacro:property name="base_to_hip_x" value="0.175" />
-    <xacro:property name="base_to_hip_y" value="0.105" />
-    <xacro:property name="hip_to_upper_leg_distance" value="0.06" />
-    <xacro:property name="upper_leg_to_lower_leg_distance" value="0.141" />
-    <xacro:property name="lower_leg_to_foot_distance" value="0.141" />
-    <xacro:property name="hip_mesh_path" value="package://champ_description/meshes/hip.stl" />
-    <xacro:property name="upper_leg_mesh_path" value="package://champ_description/meshes/upper_leg.stl" />
-    <xacro:property name="lower_leg_mesh_path" value="package://champ_description/meshes/lower_leg.stl" />
-    <material name="black">
-        <color rgba="0 0 0 0.6" />
-    </material>
-    <link name="world" />
+    <xacro:include filename="$(find champ_description)/urdf/properties.urdf.xacro" />
+    <material name="black"><color rgba="0.15 0.15 0.15 1.0" /></material>
+    <link name="champ"/>
     <link name="base_link">
+        <inertial>
+            <mass value="${base_mass}" />
+            <inertia ixx="${(1/12) * base_mass * (base_y_length * base_y_length + base_z_length * base_z_length)}" ixy="0.0" ixz="0.0"
+                     iyy="${(1/12) * base_mass * (base_x_length * base_x_length + base_z_length * base_z_length)}" iyz="0.0"
+                     izz="${(1/12) * base_mass * (base_x_length * base_x_length + base_y_length * base_y_length)}" />
+        </inertial>
+        <collision>
+            <origin xyz="0 0 0" rpy="0 0 0" />
+            <geometry>
+                <mesh filename="${base_mesh_path}" scale="0.001 0.001 0.001" />
+            </geometry>
+        </collision>
         <visual>
             <origin xyz="0 0 0" rpy="0 0 0" />
@@ -22,9 +25,19 @@
         </visual>
     </link>
-    <joint name="base_to_world" type="fixed">
-        <parent link="world" />
+    <joint name="base_to_champ" type="fixed">
+        <parent link="champ" />
         <child link="base_link" />
         <origin xyz="0 0 0" rpy="0 0 0" />
     </joint>
+    <xacro:include filename="$(find champ_description)/urdf/leg.urdf.xacro" />
+    <xacro:champ_leg leg="lf"/>
+    <xacro:champ_leg leg="lh"/>
+    <xacro:champ_leg leg="rf"/>
+    <xacro:champ_leg leg="rh"/>
+    <gazebo>
+        <plugin name="gazebo_ros_control" filename="libgazebo_ros_control.so">
+            <robotNamespace>/champ</robotNamespace>
+        </plugin>
+    </gazebo>
     <link name="lf_hip_debug_link"/>
     <joint name="lf_debug_joint" type="fixed">
@@ -51,8 +64,3 @@
         <origin xyz="-${base_to_hip_x} -${base_to_hip_y} 0" rpy="0 ${pi/2} ${pi/2}" />
     </joint>
-    <xacro:include filename="$(find champ_description)/urdf/leg.urdf.xacro" />
-    <xacro:champ_leg leg="lf"/>
-    <xacro:champ_leg leg="lh"/>
-    <xacro:champ_leg leg="rf"/>
-    <xacro:champ_leg leg="rh"/>
 </robot>

File: champ_description/urdf/leg.urdf.xacro (robot description, xacro)
@@ -19,4 +19,16 @@
         </xacro:if>
         <link name="${leg}_hip_link">
+            <inertial>
+                <mass value="${hip_mass}" />
+                <inertia ixx="${(1/12) * hip_mass * (hip_y_length * hip_y_length + hip_z_length * hip_z_length)}" ixy="0.0" ixz="0.0"
+                         iyy="${(1/12) * hip_mass * (hip_x_length * hip_x_length + hip_z_length * hip_z_length)}" iyz="0.0"
+                         izz="${(1/12) * hip_mass * (hip_x_length * hip_x_length + hip_y_length * hip_y_length)}" />
+            </inertial>
+            <collision>
+                <origin xyz="0 0 0" rpy="0 0 0" />
+                <geometry>
+                    <mesh filename="${hip_mesh_path}" scale="0.001 0.001 0.001" />
+                </geometry>
+            </collision>
             <visual>
                 <origin xyz="0 0 0" rpy="0 0 0" />
@@ -27,12 +39,17 @@
             </visual>
         </link>
-        <joint name="${leg}_hip_joint" type="revolute">
-            <axis xyz="0 1 0" />
-            <limit effort="1000.0" lower="-${pi}" upper="${pi}" velocity="0.5" />
-            <parent link="base_link" />
-            <child link="${leg}_hip_link" />
-            <origin xyz="${base_to_hip_xyz}" rpy="-${pi/2} ${pi/2} 0" />
-        </joint>
         <link name="${leg}_upper_leg_link">
+            <inertial>
+                <mass value="${upper_leg_mass}" />
+                <inertia ixx="${(1/12) * upper_leg_mass * (upper_leg_y_length * upper_leg_y_length + upper_leg_z_length * upper_leg_z_length)}" ixy="0.0" ixz="0.0"
+                         iyy="${(1/12) * upper_leg_mass * (upper_leg_x_length * upper_leg_x_length + upper_leg_z_length * upper_leg_z_length)}" iyz="0.0"
+                         izz="${(1/12) * upper_leg_mass * (upper_leg_x_length * upper_leg_x_length + upper_leg_y_length * upper_leg_y_length)}" />
+            </inertial>
+            <collision>
+                <origin xyz="0 0 0" rpy="0 0 0" />
+                <geometry>
+                    <mesh filename="${upper_leg_mesh_path}" scale="0.001 0.001 0.001" />
+                </geometry>
+            </collision>
             <visual>
                 <origin xyz="0 0 0" rpy="0 0 0" />
@@ -43,12 +60,17 @@
             </visual>
         </link>
-        <joint name="${leg}_upper_leg_joint" type="revolute">
-            <axis xyz="0 0 1" />
-            <limit effort="1000.0" lower="-${pi}" upper="${pi}" velocity="0.5" />
-            <parent link="${leg}_hip_link" />
-            <child link="${leg}_upper_leg_link" />
-            <origin xyz="0 0 ${hip_to_upper_leg}" rpy="0 0 0" />
-        </joint>
         <link name="${leg}_lower_leg_link">
+            <inertial>
+                <mass value="${lower_leg_mass}" />
+                <inertia ixx="${(1/12) * lower_leg_mass * (lower_leg_y_length * lower_leg_y_length + lower_leg_z_length * lower_leg_z_length)}" ixy="0.0" ixz="0.0"
+                         iyy="${(1/12) * lower_leg_mass * (lower_leg_x_length * lower_leg_x_length + lower_leg_z_length * lower_leg_z_length)}" iyz="0.0"
+                         izz="${(1/12) * lower_leg_mass * (lower_leg_x_length * lower_leg_x_length + lower_leg_y_length * lower_leg_y_length)}" />
+            </inertial>
+            <collision>
+                <origin xyz="0 0 0" rpy="0 0 0" />
+                <geometry>
+                    <mesh filename="${lower_leg_mesh_path}" scale="0.001 0.001 0.001" />
+                </geometry>
+            </collision>
             <visual>
                 <origin xyz="0 0 0" rpy="0 0 0" />
@@ -59,4 +81,19 @@
             </visual>
         </link>
+        <link name="${leg}_foot_link" />
+        <joint name="${leg}_hip_joint" type="revolute">
+            <axis xyz="0 1 0" />
+            <limit effort="1000.0" lower="-${pi}" upper="${pi}" velocity="0.5" />
+            <parent link="base_link" />
+            <child link="${leg}_hip_link" />
+            <origin xyz="${base_to_hip_xyz}" rpy="-${pi/2} ${pi/2} 0" />
+        </joint>
+        <joint name="${leg}_upper_leg_joint" type="revolute">
+            <axis xyz="0 0 1" />
+            <limit effort="1000.0" lower="-${pi}" upper="${pi}" velocity="0.5" />
+            <parent link="${leg}_hip_link" />
+            <child link="${leg}_upper_leg_link" />
+            <origin xyz="0 0 ${hip_to_upper_leg}" rpy="0 0 0" />
+        </joint>
         <joint name="${leg}_lower_leg_joint" type="revolute">
             <axis xyz="0 0 1" />
@@ -66,5 +103,4 @@
             <origin xyz="${upper_leg_to_lower_leg_distance} 0 0" rpy="0 0 0" />
         </joint>
-        <link name="${leg}_foot_link" />
         <joint name="${leg}_foot_joint" type="fixed">
             <parent link="${leg}_lower_leg_link" />
@@ -72,4 +108,40 @@
             <origin xyz="${lower_leg_to_foot_distance} 0 0" rpy="0 0 0" />
         </joint>
+        <transmission name="${leg}_hip_joint_trans">
+            <type>transmission_interface/SimpleTransmission</type>
+            <joint name="${leg}_hip_joint">
+                <hardwareInterface>hardware_interface/PositionJointInterface</hardwareInterface>
+                <!-- <hardwareInterface>hardware_interface/EffortJointInterface</hardwareInterface> -->
+            </joint>
+            <actuator name="${leg}_hip_joint_motor">
+                <hardwareInterface>hardware_interface/PositionJointInterface</hardwareInterface>
+                <!-- <hardwareInterface>hardware_interface/EffortJointInterface</hardwareInterface> -->
+                <mechanicalReduction>1</mechanicalReduction>
+            </actuator>
+        </transmission>
+        <transmission name="${leg}_upper_leg_joint_trans">
+            <type>transmission_interface/SimpleTransmission</type>
+            <joint name="${leg}_upper_leg_joint">
+                <hardwareInterface>hardware_interface/PositionJointInterface</hardwareInterface>
+                <!-- <hardwareInterface>hardware_interface/EffortJointInterface</hardwareInterface> -->
+            </joint>
+            <actuator name="${leg}_upper_leg_joint_motor">
+                <hardwareInterface>hardware_interface/PositionJointInterface</hardwareInterface>
+                <!-- <hardwareInterface>hardware_interface/EffortJointInterface</hardwareInterface> -->
+                <mechanicalReduction>1</mechanicalReduction>
+            </actuator>
+        </transmission>
+        <transmission name="${leg}_lower_leg_joint_trans">
+            <type>transmission_interface/SimpleTransmission</type>
+            <joint name="${leg}_lower_leg_joint">
+                <hardwareInterface>hardware_interface/PositionJointInterface</hardwareInterface>
+                <!-- <hardwareInterface>hardware_interface/EffortJointInterface</hardwareInterface> -->
+            </joint>
+            <actuator name="${leg}_lower_joint_motor">
+                <hardwareInterface>hardware_interface/PositionJointInterface</hardwareInterface>
+                <!-- <hardwareInterface>hardware_interface/EffortJointInterface</hardwareInterface> -->
+                <mechanicalReduction>1</mechanicalReduction>
+            </actuator>
+        </transmission>
     </xacro:macro>
 </robot>

Commit message: added black color material

File: champ_description/urdf/champ.urdf.xacro (robot description, xacro)
@@ -6,4 +6,5 @@
     <link name="base_link">
         <inertial>
+            <origin xyz="0.065 0 0" />
             <mass value="${base_mass}" />
             <inertia ixx="${(1/12) * base_mass * (base_y_length * base_y_length + base_z_length * base_z_length)}" ixy="0.0" ixz="0.0"
@@ -25,4 +26,7 @@
         </visual>
     </link>
+    <gazebo reference="base_link">
+        <material>Gazebo/FlatBlack</material>
+    </gazebo>
     <joint name="base_to_champ" type="fixed">
         <parent link="champ" />
@@ -38,4 +42,5 @@
         <plugin name="gazebo_ros_control" filename="libgazebo_ros_control.so">
             <robotNamespace>/champ</robotNamespace>
+            <legacyModeNS>true</legacyModeNS>
         </plugin>
     </gazebo>

Commit message: shifted back cog to center

File: champ_description/urdf/champ.urdf.xacro (robot description, xacro)
@@ -6,5 +6,5 @@
     <link name="base_link">
         <inertial>
-            <origin xyz="0.065 0 0" />
+            <origin xyz="0 0 0" />
             <mass value="${base_mass}" />
             <inertia ixx="${(1/12) * base_mass * (base_y_length * base_y_length + base_z_length * base_z_length)}" ixy="0.0" ixz="0.0"

Commit message: changed from position_controller to effort_controller

File: champ_description/urdf/champ.urdf.xacro (robot description, xacro)
@@ -6,5 +6,5 @@
     <link name="base_link">
         <inertial>
-            <origin xyz="0 0 0" />
+            <origin xyz="0.075 0 0" />
             <mass value="${base_mass}" />
             <inertia ixx="${(1/12) * base_mass * (base_y_length * base_y_length + base_z_length * base_z_length)}" ixy="0.0" ixz="0.0"

File: champ_description/urdf/leg.urdf.xacro (robot description, xacro)
@@ -90,10 +90,4 @@
         </link>
         <gazebo reference="${leg}_lower_leg_link">
-            <kp>100000.0</kp>
-            <kd>100000.0</kd>
-            <mu1>1.5</mu1>
-            <mu2>1.5</mu2>
-            <fdir>1 0 0</fdir>
-            <maxVel>0.5</maxVel>
             <minDepth>0.001</minDepth>
             <material>Gazebo/FlatBlack</material>
@@ -129,11 +123,9 @@
             <type>transmission_interface/SimpleTransmission</type>
             <joint name="${leg}_hip_joint">
-                <hardwareInterface>hardware_interface/PositionJointInterface</hardwareInterface>
-                <!-- <hardwareInterface>hardware_interface/EffortJointInterface</hardwareInterface> -->
+                <hardwareInterface>hardware_interface/EffortJointInterface</hardwareInterface>
             </joint>
             <actuator name="${leg}_hip_joint_motor">
-                <hardwareInterface>hardware_interface/PositionJointInterface</hardwareInterface>
-                <!-- <hardwareInterface>hardware_interface/EffortJointInterface</hardwareInterface> -->
-                <!-- <mechanicalReduction>1</mechanicalReduction> -->
+                <hardwareInterface>hardware_interface/EffortJointInterface</hardwareInterface>
+                <mechanicalReduction>1</mechanicalReduction>
             </actuator>
         </transmission>
@@ -141,11 +133,9 @@
             <type>transmission_interface/SimpleTransmission</type>
             <joint name="${leg}_upper_leg_joint">
-                <hardwareInterface>hardware_interface/PositionJointInterface</hardwareInterface>
-                <!-- <hardwareInterface>hardware_interface/EffortJointInterface</hardwareInterface> -->
+                <hardwareInterface>hardware_interface/EffortJointInterface</hardwareInterface>
             </joint>
             <actuator name="${leg}_upper_leg_joint_motor">
-                <hardwareInterface>hardware_interface/PositionJointInterface</hardwareInterface>
-                <!-- <hardwareInterface>hardware_interface/EffortJointInterface</hardwareInterface> -->
-                <!-- <mechanicalReduction>1</mechanicalReduction> -->
+                <hardwareInterface>hardware_interface/EffortJointInterface</hardwareInterface>
+                <mechanicalReduction>1</mechanicalReduction>
             </actuator>
         </transmission>
@@ -153,11 +143,9 @@
             <type>transmission_interface/SimpleTransmission</type>
             <joint name="${leg}_lower_leg_joint">
-                <hardwareInterface>hardware_interface/PositionJointInterface</hardwareInterface>
-                <!-- <hardwareInterface>hardware_interface/EffortJointInterface</hardwareInterface> -->
+                <hardwareInterface>hardware_interface/EffortJointInterface</hardwareInterface>
             </joint>
             <actuator name="${leg}_lower_joint_motor">
-                <hardwareInterface>hardware_interface/PositionJointInterface</hardwareInterface>
-                <!-- <hardwareInterface>hardware_interface/EffortJointInterface</hardwareInterface> -->
-                <!-- <mechanicalReduction>1</mechanicalReduction> -->
+                <hardwareInterface>hardware_interface/EffortJointInterface</hardwareInterface>
+                <mechanicalReduction>1</mechanicalReduction>
             </actuator>
         </transmission>

Commit message: shift COG more to the center to prevent robot from tipping over on faster speeds

File: champ_description/urdf/champ.urdf.xacro (robot description, xacro)
@@ -6,5 +6,5 @@
     <link name="base_link">
         <inertial>
-            <origin xyz="0.075 0 0" />
+            <origin xyz="0.04 0 0" />
             <mass value="${base_mass}" />
             <inertia ixx="${(1/12) * base_mass * (base_y_length * base_y_length + base_z_length * base_z_length)}" ixy="0.0" ixz="0.0"

Commit message: renamed champ to champ_footprint

File: champ_description/urdf/champ.urdf.xacro (robot description, xacro)
@@ -3,5 +3,5 @@
     <xacro:include filename="$(find champ_description)/urdf/properties.urdf.xacro" />
     <material name="black"><color rgba="0.15 0.15 0.15 1.0" /></material>
-    <link name="champ"/>
+    <link name="champ_footprint"/>
     <link name="base_link">
         <inertial>
@@ -30,5 +30,5 @@
     </gazebo>
     <joint name="base_to_champ" type="fixed">
-        <parent link="champ" />
+        <parent link="champ_footprint" />
         <child link="base_link" />
         <origin xyz="0 0 0" rpy="0 0 0" />
@@ -79,5 +79,5 @@
         </plugin>
     </gazebo>
-    <xacro:include filename="$(find common_sensors)/urdf/sensors/kinect.urdf.xacro" />
+    <!-- <xacro:include filename="$(find common_sensors)/urdf/sensors/kinect.urdf.xacro" />
     <xacro:sensor_kinect parent="base_link">
         <property name="cam_px" value="0.23" />
@@ -87,4 +87,15 @@
         <property name="cam_op" value="0.0" />
         <property name="cam_oy" value="0.0"/>
-    </xacro:sensor_kinect>
+    </xacro:sensor_kinect> -->
+    <xacro:include filename="$(find common_sensors)/urdf/sensors/hokuyo_utm30lx.urdf.xacro" />
+    <xacro:hokuyo_utm30lx
+        name="hokuyo"
+        parent="base_link"
+        ros_topic="scan"
+        update_rate="30"
+        ray_count="1040"
+        min_angle="130"
+        max_angle="-130" >
+        <origin xyz="0.0 0.0 0.12" rpy="0 0 0"/>
+    </xacro:hokuyo_utm30lx>
 </robot>

Commit message: fine tuned leg speed and effort

File: champ_description/urdf/champ.urdf.xacro (robot description, xacro)
@@ -6,5 +6,5 @@
     <link name="base_link">
         <inertial>
-            <origin xyz="0.04 0 0" />
+            <origin xyz="0 0 0" />
             <mass value="${base_mass}" />
             <inertia ixx="${(1/12) * base_mass * (base_y_length * base_y_length + base_z_length * base_z_length)}" ixy="0.0" ixz="0.0"

File: champ_description/urdf/leg.urdf.xacro (robot description, xacro)
@@ -69,5 +69,5 @@
         <link name="${leg}_lower_leg_link">
             <inertial>
-                <origin xyz="0.065 0 0" />
+                <origin xyz="0.065 0.005 0" />
                 <mass value="${lower_leg_mass}" />
                 <inertia ixx="${(1/12) * lower_leg_mass * (lower_leg_y_length * lower_leg_y_length + lower_leg_z_length * lower_leg_z_length)}" ixy="0.0" ixz="0.0"
@@ -101,5 +101,5 @@
         <joint name="${leg}_hip_joint" type="revolute">
             <axis xyz="0 1 0" />
-            <limit effort="20" lower="-${pi}" upper="${pi}" velocity="2.0" />
+            <limit effort="25" lower="-${pi}" upper="${pi}" velocity="1.5" />
             <parent link="base_link" />
             <child link="${leg}_hip_link" />
@@ -108,5 +108,5 @@
         <joint name="${leg}_upper_leg_joint" type="revolute">
             <axis xyz="0 0 1" />
-            <limit effort="20" lower="-${pi}" upper="${pi}" velocity="2.0" />
+            <limit effort="25" lower="-${pi}" upper="${pi}" velocity="1.5" />
             <parent link="${leg}_hip_link" />
             <child link="${leg}_upper_leg_link" />
@@ -115,5 +115,5 @@
         <joint name="${leg}_lower_leg_joint" type="revolute">
             <axis xyz="0 0 1" />
-            <limit effort="20" lower="-${pi}" upper="${pi}" velocity="2.0" />
+            <limit effort="25" lower="-${pi}" upper="${pi}" velocity="1.5" />
             <parent link="${leg}_upper_leg_link" />
             <child link="${leg}_lower_leg_link" />

File: champ_description/urdf/properties.urdf.xacro (robot description, xacro)
@@ -7,5 +7,5 @@
     <xacro:property name="lower_leg_to_foot_distance" value="0.141" />
     <xacro:property name="hip_mesh_path" value="package://champ_description/meshes/hip.stl" />
-    <xacro:property name="hip_mass" value="0.25" />
+    <xacro:property name="hip_mass" value="0.250" />
     <xacro:property name="hip_x_length" value="0.130" />
     <xacro:property name="hip_y_length" value="0.112" />
@@ -17,5 +17,5 @@
     <xacro:property name="upper_leg_z_length" value="0.03" />
     <xacro:property name="lower_leg_mesh_path" value="package://champ_description/meshes/lower_leg.stl" />
-    <xacro:property name="lower_leg_mass" value="0.25" />
+    <xacro:property name="lower_leg_mass" value="0.125" />
     <xacro:property name="lower_leg_x_length" value="0.156" />
     <xacro:property name="lower_leg_y_length" value="0.039" />

Commit message: changed hardcoded values to paramertized ones

File: champ_description/urdf/champ.urdf.xacro (robot description, xacro)
@@ -30,5 +30,5 @@
     </gazebo>
     <joint name="base_to_champ" type="fixed">
-        <parent link="champ_footprint" />
+        <parent link="base_footprint" />
         <child link="base_link" />
         <origin xyz="0 0 0" rpy="0 0 0" />
@@ -97,5 +97,5 @@
         min_angle="130"
         max_angle="-130" >
-        <origin xyz="0.0 0.0 0.12" rpy="0 0 0"/>
+        <origin xyz="0.0 0.0 ${base_z_length / 2 + 0.04}" rpy="0 0 0"/>
     </xacro:hokuyo_utm30lx>
 </robot>

File: champ_description/urdf/leg.urdf.xacro (robot description, xacro)
@@ -44,5 +44,5 @@
         <link name="${leg}_upper_leg_link">
             <inertial>
-                <origin xyz="0.065 0 0" />
+                <origin xyz="${(upper_leg_x_length / 2) - ((upper_leg_x_length - upper_leg_to_lower_leg_distance) / 2)} 0 0" />
                 <mass value="${upper_leg_mass}" />
                 <inertia ixx="${(1/12) * upper_leg_mass * (upper_leg_y_length * upper_leg_y_length + upper_leg_z_length * upper_leg_z_length)}" ixy="0.0" ixz="0.0"
@@ -69,5 +69,5 @@
         <link name="${leg}_lower_leg_link">
             <inertial>
-                <origin xyz="0.065 0.005 0" />
+                <origin xyz="${(lower_leg_to_foot_distance - (lower_leg_x_length - lower_leg_to_foot_distance)) / 2} 0 0" />
                 <mass value="${lower_leg_mass}" />
                 <inertia ixx="${(1/12) * lower_leg_mass * (lower_leg_y_length * lower_leg_y_length + lower_leg_z_length * lower_leg_z_length)}" ixy="0.0" ixz="0.0"

Commit message: renamed champ_footprint to base_footprint

File: champ_description/urdf/champ.urdf.xacro (robot description, xacro)
@@ -3,5 +3,5 @@
     <xacro:include filename="$(find champ_description)/urdf/properties.urdf.xacro" />
     <material name="black"><color rgba="0.15 0.15 0.15 1.0" /></material>
-    <link name="champ_footprint"/>
+    <link name="base_footprint"/>
     <link name="base_link">
         <inertial>
