Commit message: added imu plugin

File: champ_description/urdf/champ.urdf.xacro (robot description, xacro)
@@ -29,8 +29,19 @@
         <material>Gazebo/FlatBlack</material>
     </gazebo>
-    <joint name="base_to_champ" type="fixed">
+    <joint name="base_to_footprint" type="fixed">
         <parent link="base_footprint" />
         <child link="base_link" />
         <origin xyz="0 0 0" rpy="0 0 0" />
+    </joint>
+    <link name="imu_link">
+        <inertial>
+            <mass value="0.001"/>
+            <origin xyz="0 0 0" rpy="0 0 0"/>
+            <inertia ixx="1e-09" ixy="0.0" ixz="0.0" iyy="1e-09" iyz="0.0" izz="1e-09"/>
+        </inertial>
+    </link>
+        <joint name="imu_joint" type="fixed">
+        <parent link="base_link" />
+        <child link="imu_link" />
     </joint>
     <xacro:include filename="$(find champ_description)/urdf/leg.urdf.xacro" />
@@ -88,15 +99,18 @@
             <legacyModeNS>true</legacyModeNS>
         </plugin>
-        <plugin name="p3d_base_controller" filename="libgazebo_ros_p3d.so">
-            <alwaysOn>true</alwaysOn>
-            <updateRate>10.0</updateRate>
-            <bodyName>base_link</bodyName>
-            <topicName>odom/ground_truth</topicName>
-            <gaussianNoise>0.01</gaussianNoise>
-            <frameName>world</frameName>
-            <xyzOffsets>0 0 0</xyzOffsets>
-            <rpyOffsets>0 0 0</rpyOffsets>
+    </gazebo>
+    <gazebo>
+        <plugin name="imu_controller" filename="libhector_gazebo_ros_imu.so">
+            <robotNamespace>/</robotNamespace>
+            <updateRate>50.0</updateRate>
+            <bodyName>imu_link</bodyName>
+            <topicName>imu/data</topicName>
+            <accelDrift>0.005 0.005 0.005</accelDrift>
+            <accelGaussianNoise>0.005 0.005 0.005</accelGaussianNoise>
+            <rateDrift>0.005 0.005 0.005 </rateDrift>
+            <rateGaussianNoise>0.005 0.005 0.005 </rateGaussianNoise>
+            <headingDrift>0.005</headingDrift>
+            <headingGaussianNoise>0.005</headingGaussianNoise>
         </plugin>
-        <plugin name="contact_plugin" filename="libcontact.so"/>
     </gazebo>
 </robot>

Commit message: added depth sensor

File: champ_description/urdf/champ.urdf.xacro (robot description, xacro)
@@ -74,13 +74,4 @@
         <origin xyz="-${base_to_hip_x} -${base_to_hip_y} 0" rpy="0 ${pi/2} ${pi/2}" />
     </joint>
-    <!-- <xacro:include filename="$(find common_sensors)/urdf/sensors/kinect.urdf.xacro" />
-    <xacro:sensor_kinect parent="base_link">
-        <property name="cam_px" value="0.23" />
-        <property name="cam_py" value="0.0" />
-        <property name="cam_pz" value="0.115" />
-        <property name="cam_or" value="0.0" />
-        <property name="cam_op" value="0.0" />
-        <property name="cam_oy" value="0.0"/>
-    </xacro:sensor_kinect> -->
     <xacro:include filename="$(find common_sensors)/urdf/sensors/hokuyo_utm30lx.urdf.xacro" />
     <xacro:hokuyo_utm30lx
@@ -94,10 +85,16 @@
         <origin xyz="0.0 0.0 ${base_z_length / 2 + 0.04}" rpy="0 0 0"/>
     </xacro:hokuyo_utm30lx>
-    <gazebo>
-        <plugin name="gazebo_ros_control" filename="libgazebo_ros_control.so">
-            <robotNamespace>/champ</robotNamespace>
-            <legacyModeNS>true</legacyModeNS>
-        </plugin>
-    </gazebo>
+    <gazebo reference="hokuyo_frame">
+		<material>Gazebo/FlatBlack</material>
+	</gazebo>
+    <xacro:include filename="$(find common_sensors)/urdf/sensors/xtion.urdf.xacro" />
+    <xacro:sensor_xtion
+        parent="base_link"
+        camera_name="camera">
+        <origin xyz="${base_x_length / 2} 0.0 ${base_z_length / 2 + 0.01}" rpy="0 0 0"/>
+    </xacro:sensor_xtion>
+    <gazebo reference="hokuyo_frame">
+		<material>Gazebo/FlatBlack</material>
+	</gazebo>
     <gazebo>
         <plugin name="imu_controller" filename="libhector_gazebo_ros_imu.so">
@@ -114,3 +111,9 @@
         </plugin>
     </gazebo>
+    <gazebo>
+        <plugin name="gazebo_ros_control" filename="libgazebo_ros_control.so">
+            <robotNamespace>/champ</robotNamespace>
+            <legacyModeNS>true</legacyModeNS>
+        </plugin>
+    </gazebo>
 </robot>

Commit message: omitted fixed transform betwoon base_footprint and base_link

File: champ_description/urdf/champ.urdf.xacro (robot description, xacro)
@@ -3,5 +3,4 @@
     <xacro:include filename="$(find champ_description)/urdf/properties.urdf.xacro" />
     <material name="black"><color rgba="0.15 0.15 0.15 1.0" /></material>
-    <link name="base_footprint"/>
     <link name="base_link">
         <inertial>
@@ -29,9 +28,4 @@
         <material>Gazebo/FlatBlack</material>
     </gazebo>
-    <joint name="base_to_footprint" type="fixed">
-        <parent link="base_footprint" />
-        <child link="base_link" />
-        <origin xyz="0 0 0" rpy="0 0 0" />
-    </joint>
     <link name="imu_link">
         <inertial>

Commit message: added odometry ground truth plugin

File: champ_description/urdf/champ.urdf.xacro (robot description, xacro)
@@ -3,4 +3,5 @@
     <xacro:include filename="$(find champ_description)/urdf/properties.urdf.xacro" />
     <material name="black"><color rgba="0.15 0.15 0.15 1.0" /></material>
+    <!-- <link name="champ"/> -->
     <link name="base_link">
         <inertial>
@@ -25,4 +26,8 @@
         </visual>
     </link>
+    <!-- <joint name="base_champ_joint" type="fixed">
+        <parent link="champ" />
+        <child link="base_link" />
+    </joint> -->
     <gazebo reference="base_link">
         <material>Gazebo/FlatBlack</material>
@@ -35,5 +40,5 @@
         </inertial>
     </link>
-        <joint name="imu_joint" type="fixed">
+    <joint name="imu_joint" type="fixed">
         <parent link="base_link" />
         <child link="imu_link" />
@@ -106,4 +111,16 @@
     </gazebo>
     <gazebo>
+      <plugin name="p3d_base_controller" filename="libgazebo_ros_p3d.so">
+            <alwaysOn>true</alwaysOn>
+            <updateRate>10.0</updateRate>
+            <bodyName>base_link</bodyName>
+            <topicName>odom/ground_truth</topicName>
+            <gaussianNoise>0.01</gaussianNoise>
+            <frameName>world</frameName>
+            <xyzOffsets>0 0 0</xyzOffsets>
+            <rpyOffsets>0 0 0</rpyOffsets>
+        </plugin>
+    </gazebo>
+    <gazebo>
         <plugin name="gazebo_ros_control" filename="libgazebo_ros_control.so">
             <robotNamespace>/champ</robotNamespace>

Commit message: shifted hip debug links to leg urdf

File: champ_description/urdf/champ.urdf.xacro (robot description, xacro)
@@ -49,28 +49,4 @@
     <xacro:champ_leg leg="rf"/>
     <xacro:champ_leg leg="rh"/>
-    <link name="lf_hip_debug_link"/>
-    <joint name="lf_debug_joint" type="fixed">
-        <parent link="base_link" />
-        <child link="lf_hip_debug_link" />
-        <origin xyz="${base_to_hip_x} ${base_to_hip_y} 0" rpy="0 ${pi/2} ${pi/2}" />
-    </joint>
-    <link name="rf_hip_debug_link"/>
-    <joint name="rf_debug_joint" type="fixed">
-        <parent link="base_link" />
-        <child link="rf_hip_debug_link" />
-        <origin xyz="${base_to_hip_x} -${base_to_hip_y} 0" rpy="0 ${pi/2} ${pi/2}" />
-    </joint>
-    <link name="lh_hip_debug_link"/>
-    <joint name="lh_debug_joint" type="fixed">
-        <parent link="base_link" />
-        <child link="lh_hip_debug_link" />
-        <origin xyz="-${base_to_hip_x} ${base_to_hip_y} 0" rpy="0 ${pi/2} ${pi/2}" />
-    </joint>
-    <link name="rh_hip_debug_link"/>
-    <joint name="rh_debug_joint" type="fixed">
-        <parent link="base_link" />
-        <child link="rh_hip_debug_link" />
-        <origin xyz="-${base_to_hip_x} -${base_to_hip_y} 0" rpy="0 ${pi/2} ${pi/2}" />
-    </joint>
     <xacro:include filename="$(find common_sensors)/urdf/sensors/hokuyo_utm30lx.urdf.xacro" />
     <xacro:hokuyo_utm30lx

File: champ_description/urdf/leg.urdf.xacro (robot description, xacro)
@@ -18,4 +18,5 @@
             <xacro:property name="hip_to_upper_leg" value="-${hip_to_upper_leg_distance}" />
         </xacro:if>
+        <link name="${leg}_hip_debug_link"/>
         <link name="${leg}_hip_link">
             <inertial>
@@ -99,4 +100,9 @@
         </gazebo>
         <link name="${leg}_foot_link" />
+        <joint name="${leg}_debug_joint" type="fixed">
+            <parent link="base_link" />
+            <child link="${leg}_hip_debug_link" />
+            <origin xyz="${base_to_hip_xyz}" rpy="0 ${pi/2} ${pi/2}" />
+        </joint>
         <joint name="${leg}_hip_joint" type="revolute">
             <axis xyz="0 1 0" />

Commit message: shift com more to the front

File: champ_description/urdf/champ.urdf.xacro (robot description, xacro)
@@ -6,5 +6,5 @@
     <link name="base_link">
         <inertial>
-            <origin xyz="0 0 0" />
+            <origin xyz="0.02 0 0" />
             <mass value="${base_mass}" />
             <inertia ixx="${(1/12) * base_mass * (base_y_length * base_y_length + base_z_length * base_z_length)}" ixy="0.0" ixz="0.0"

Commit message: fixed base inertia

File: champ_description/urdf/champ.urdf.xacro (robot description, xacro)
@@ -6,5 +6,5 @@
     <link name="base_link">
         <inertial>
-            <origin xyz="0.02 0 0" />
+            <origin xyz="0 0 0" />
             <mass value="${base_mass}" />
             <inertia ixx="${(1/12) * base_mass * (base_y_length * base_y_length + base_z_length * base_z_length)}" ixy="0.0" ixz="0.0"

Commit message: Added and tuned effort controller for joints

File: champ_description/urdf/champ.urdf.xacro (robot description, xacro)
@@ -13,5 +13,5 @@
             <origin xyz="0 0 0" rpy="0 0 0" />
             <geometry>
-                <mesh filename="file://$(find champ_description)/meshes/base.stl" scale="0.001 0.001 0.001" />
+                <mesh filename="file://$(find champ_description)/meshes/base_simple.stl" scale="0.001 0.001 0.001" />
             </geometry>
             <material name="black" />
@@ -32,19 +32,24 @@
         <origin rpy="0 0 0" xyz="0 0 0"/>
     </joint>
+    <!-- <link name="world"/>
+    <joint name="fixed" type="fixed">
+        <parent link="world"/>
+        <child link="base_link"/>
+      </joint> -->
     <gazebo reference="base_link">
         <material>Gazebo/FlatBlack</material>
     </gazebo>
     <xacro:include filename="$(find champ_description)/urdf/leg.urdf.xacro" />
-    <xacro:include filename="$(find champ_description)/urdf/accessories.urdf.xacro" />
-    <xacro:accessories
+    <!-- <xacro:include filename="$(find champ_description)/urdf/accessories.urdf.xacro" /> -->
+    <!-- <xacro:accessories
         base_name="base_link"
         base_length="${base_x_length}"
         base_height="${base_z_length}"
-    />
+    /> -->
     <xacro:champ_leg leg="lf"/>
     <xacro:champ_leg leg="lh"/>
     <xacro:champ_leg leg="rf"/>
     <xacro:champ_leg leg="rh"/>
-    <gazebo>
+    <!-- <gazebo>
       <plugin name="p3d_base_controller" filename="libgazebo_ros_p3d.so">
             <ros>
@@ -59,5 +64,5 @@
             <gaussian_noise>0.01</gaussian_noise>
     </plugin>
-    </gazebo>
+    </gazebo> -->
     <gazebo>
     <plugin filename="libgazebo_ros2_control.so" name="gazebo_ros2_control">
@@ -67,3 +72,8 @@
       </plugin>
     </gazebo>
+    <!-- <gazebo>
+        <plugin filename="ign_ros2_control-system" name="ign_ros2_control::IgnitionROS2ControlPlugin">
+            <parameters>$(find champ_gazebo)/config/ros_control.yaml</parameters>
+          </plugin>
+    </gazebo> -->
 </robot>

File: champ_description/urdf/leg.urdf.xacro (robot description, xacro)
@@ -90,13 +90,4 @@
             </visual>
         </link>
-        <gazebo reference="${leg}_lower_leg_link">
-            <kp>1000000.0</kp>
-            <kd>1.0</kd>
-            <mu1>0.8</mu1>
-            <mu2>0.8</mu2>
-            <maxVel>0.0</maxVel>
-            <minDepth>0.001</minDepth>
-            <material>Gazebo/FlatBlack</material>
-        </gazebo>
         <link name="${leg}_foot_link" />
         <joint name="${leg}_debug_joint" type="fixed">
@@ -134,39 +125,20 @@
         <ros2_control name="${leg}_hip" type="system">
             <hardware>
-              <plugin>gazebo_ros2_control/GazeboSystem</plugin>
+                <plugin>gazebo_ros2_control/GazeboSystem</plugin>
             </hardware>
             <joint name="${leg}_hip_joint">
-                <!-- <command_interface name="effort">
-                    <param name="min">-1000</param>
-                    <param name="max">1000</param>
-                </command_interface>
+                <command_interface name="effort"/>
                 <state_interface name="position"/>
                 <state_interface name="velocity"/>
-                <state_interface name="effort"/> -->
-                <command_interface name="position">
-                    <param name="min">-55</param>
-                    <param name="max">55</param>
-                </command_interface>
-                <state_interface name="position">
-                <param name="initial_value">1.0</param>
-                </state_interface>
-                <state_interface name="velocity"/>
-                <state_interface name="effort"/>
             </joint>
         </ros2_control>
         <ros2_control name="${leg}_upper_leg" type="system">
             <hardware>
-              <plugin>gazebo_ros2_control/GazeboSystem</plugin>
+                <plugin>gazebo_ros2_control/GazeboSystem</plugin>
             </hardware>
             <joint name="${leg}_upper_leg_joint">
-                <command_interface name="position">
-                    <param name="min">-55</param>
-                    <param name="max">55</param>
-                </command_interface>
-                <state_interface name="position">
-                <param name="initial_value">1.0</param>
-                </state_interface>
+                <command_interface name="effort"/>
+                <state_interface name="position"/>
                 <state_interface name="velocity"/>
-                <state_interface name="effort"/>
             </joint>
         </ros2_control>
@@ -176,13 +148,7 @@
             </hardware>
             <joint name="${leg}_lower_leg_joint">
-                <command_interface name="position">
-                    <param name="min">-55</param>
-                    <param name="max">55</param>
-                </command_interface>
-                <state_interface name="position">
-                <param name="initial_value">1.0</param>
-                </state_interface>
+                <command_interface name="effort"/>
+                <state_interface name="position"/>
                 <state_interface name="velocity"/>
-                <state_interface name="effort"/>
             </joint>
         </ros2_control>

File: champ_description/urdf/properties.urdf.xacro (robot description, xacro)
@@ -11,15 +11,15 @@
     <xacro:property name="hip_y_length" value="0.08" />
     <xacro:property name="hip_z_length" value="0.130" />
-    <xacro:property name="upper_leg_mesh_path" value="file://$(find champ_description)/meshes/upper_leg.stl" />
+    <xacro:property name="upper_leg_mesh_path" value="file://$(find champ_description)/meshes/upper_leg_simple.stl" />
     <xacro:property name="upper_leg_mass" value="0.125" />
     <xacro:property name="upper_leg_x_length" value="0.05" />
     <xacro:property name="upper_leg_y_length" value="0.03" />
     <xacro:property name="upper_leg_z_length" value="0.1905" />
-    <xacro:property name="lower_leg_mesh_path" value="file://$(find champ_description)/meshes/lower_leg.stl" />
+    <xacro:property name="lower_leg_mesh_path" value="file://$(find champ_description)/meshes/lower_leg_simple.stl" />
     <xacro:property name="lower_leg_mass" value="0.125" />
     <xacro:property name="lower_leg_x_length" value="0.039" />
     <xacro:property name="lower_leg_y_length" value="0.022" />
     <xacro:property name="lower_leg_z_length" value="0.156" />
-    <xacro:property name="base_mesh_path" value="file://$(find champ_description)/meshes/base.stl" />
+    <xacro:property name="base_mesh_path" value="file://$(find champ_description)/meshes/base_simple.stl" />
     <xacro:property name="base_mass" value="2.0" />
     <xacro:property name="base_x_length" value="0.5" />

Commit message: Working demo in rviz

File: champ_description/urdf/champ.urdf.xacro (robot description, xacro)
@@ -41,15 +41,15 @@
     </gazebo>
     <xacro:include filename="$(find champ_description)/urdf/leg.urdf.xacro" />
-    <!-- <xacro:include filename="$(find champ_description)/urdf/accessories.urdf.xacro" /> -->
-    <!-- <xacro:accessories
+    <xacro:include filename="$(find champ_description)/urdf/accessories.urdf.xacro" />
+    <xacro:accessories
         base_name="base_link"
         base_length="${base_x_length}"
         base_height="${base_z_length}"
-    /> -->
+    />
     <xacro:champ_leg leg="lf"/>
     <xacro:champ_leg leg="lh"/>
     <xacro:champ_leg leg="rf"/>
     <xacro:champ_leg leg="rh"/>
-    <!-- <gazebo>
+    <gazebo>
       <plugin name="p3d_base_controller" filename="libgazebo_ros_p3d.so">
             <ros>
@@ -64,9 +64,7 @@
             <gaussian_noise>0.01</gaussian_noise>
     </plugin>
-    </gazebo> -->
+    </gazebo>
     <gazebo>
     <plugin filename="libgazebo_ros2_control.so" name="gazebo_ros2_control">
-        <!-- <robot_param>/robot_description</robot_param>
-        <robot_param_node>/robot_state_publisher</robot_param_node> -->
         <parameters>$(find champ_gazebo)/config/ros_control.yaml</parameters>
       </plugin>

File: champ_description/urdf/hokuyo_utm30lx.urdf.xacro (robot description, xacro)
@@ -17,5 +17,5 @@
           <origin xyz="0 0 0" rpy="0 0 0" />
           <geometry>
-          <mesh filename="file://$(find champ_description)/meshes/hokuyo_utm30lx/hokuyo_utm_30lx$(optenv TEST_SELF_FILTER).dae"/>
+          <mesh filename="file://$(find champ_description)/meshes/hokuyo_utm_30lx$(optenv TEST_SELF_FILTER).dae"/>
         </geometry>
         </visual>

File: champ_description/urdf/leg.urdf.xacro (robot description, xacro)
@@ -90,5 +90,15 @@
             </visual>
         </link>
+        <gazebo reference="${leg}_lower_leg_link">
+            <kp>1000000.0</kp>
+            <kd>1.0</kd>
+            <mu1>0.8</mu1>
+            <mu2>0.8</mu2>
+            <maxVel>0.0</maxVel>
+            <minDepth>0.001</minDepth>
+            <material>Gazebo/FlatBlack</material>
+        </gazebo>
         <link name="${leg}_foot_link" />
+        <!-- <link name="${leg}_foot_link_debug" /> -->
         <joint name="${leg}_debug_joint" type="fixed">
             <parent link="base_link" />
@@ -120,7 +130,12 @@
             <parent link="${leg}_lower_leg_link" />
             <child link="${leg}_foot_link" />
-            <!-- <origin xyz="0.00325 0 -${lower_leg_to_foot_distance}" rpy="0 0 0" /> -->
-            <origin xyz="0 0 -${lower_leg_to_foot_distance}" rpy="0 0 0" />
+            <origin xyz="0.00325 0 -${lower_leg_to_foot_distance}" rpy="0 0 0" />
+            <!-- <origin xyz="0 0 -${lower_leg_to_foot_distance}" rpy="0 0 0" /> -->
         </joint>
+        <!-- <joint name="${leg}_debug_joint_foot" type="fixed">
+            <parent link="${leg}_foot_link" />
+            <child link="${leg}_foot_link_debug" />
+            <origin xyz="0 0 0" rpy="0 0 0" />
+        </joint> -->
         <ros2_control name="${leg}_hip" type="system">
             <hardware>
