Commit message: renamed xml namespace to newer ones

File: champ_description/urdf/accessories.urdf.xacro (robot description, xacro)
@@ -1,4 +1,4 @@
 <?xml version="1.0"?>
-<robot xmlns:xacro="http://www.ros.org/wiki/xacro">
+<robot xmlns:xacro="http://ros.org/wiki/xacro">
     <xacro:include filename="$(find common_sensors)/urdf/sensors/hokuyo_utm30lx.urdf.xacro" />
     <xacro:include filename="$(find common_sensors)/urdf/sensors/xtion.urdf.xacro" />

File: champ_description/urdf/champ.urdf (robot description, URDF)
Before this commit: robot champ, 21 links, 20 joints
Links:
- added link camera_base_frame, mass 0.001
- added link camera_depth_frame, mass 0.01
- added link camera_depth_optical_frame, mass 0.001
- added link camera_link, mass 0.01; collision box size=0.15 0.05 0.07; visual mesh filename=package://common_sensors/meshes/sensors/asus_xtion_pro_live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 scale=0.001 0.001 0.001
- added link camera_rgb_frame, mass 0.001
- added link camera_rgb_optical_frame, mass 0.001
- added link imu_link, mass 0.001
Joints:
- added joint camera_base_joint: type fixed, parent base_link, child camera_base_frame, origin xyz=0.25 0.0 0.075 rpy=0 0 0
- added joint camera_depth_joint: type fixed, parent camera_base_frame, child camera_depth_frame, origin xyz=0 0.0499 0 rpy=0 0 0
- added joint camera_depth_optical_joint: type fixed, parent camera_depth_frame, child camera_depth_optical_frame, origin xyz=0 0 0 rpy=-1.57079632679 0 -1.57079632679
- added joint camera_joint: type fixed, parent camera_base_frame, child camera_link, origin xyz=0 0 0 rpy=0 0 0
- added joint camera_rgb_joint: type fixed, parent camera_base_frame, child camera_rgb_frame, origin xyz=0 0.022 0 rpy=0 0 0
- added joint camera_rgb_optical_joint: type fixed, parent camera_rgb_frame, child camera_rgb_optical_frame, origin xyz=0 0 0 rpy=-1.57079632679 0 -1.57079632679
- added joint imu_joint: type fixed, parent base_link, child imu_link

File: champ_description/urdf/champ.urdf.xacro (robot description, xacro)
@@ -1,4 +1,4 @@
 <?xml version="1.0"?>
-<robot name="champ" xmlns:xacro="http://www.ros.org/wiki/xacro">
+<robot name="champ" xmlns:xacro="http://ros.org/wiki/xacro">
     <xacro:include filename="$(find champ_description)/urdf/properties.urdf.xacro" />
     <material name="black"><color rgba="0.15 0.15 0.15 1.0" /></material>
@@ -34,7 +34,5 @@
     </gazebo>
     <xacro:include filename="$(find champ_description)/urdf/leg.urdf.xacro" />
-    <xacro:if value="$(optenv ENABLE_SENSORS 0)">
-        <xacro:include filename="$(find champ_description)/urdf/accessories.urdf.xacro" />
-    </xacro:if>
+    <xacro:include filename="$(find champ_description)/urdf/accessories.urdf.xacro" />
     <xacro:champ_leg leg="lf"/>
     <xacro:champ_leg leg="lh"/>

File: champ_description/urdf/leg.urdf.xacro (robot description, xacro)
@@ -1,4 +1,4 @@
 <?xml version="1.0"?>
-<robot xmlns:xacro="http://www.ros.org/wiki/xacro">
+<robot xmlns:xacro="http://ros.org/wiki/xacro">
     <xacro:macro name="champ_leg" params="leg  " >
         <xacro:if value="${leg == 'lf'}">

File: champ_description/urdf/properties.urdf.xacro (robot description, xacro)
@@ -1,4 +1,4 @@
 <?xml version="1.0"?>
-<robot xmlns:xacro="http://www.ros.org/wiki/xacro">
+<robot xmlns:xacro="http://ros.org/wiki/xacro">
     <xacro:property name="base_to_hip_x" value="0.175" />
     <xacro:property name="base_to_hip_y" value="0.105" />

Commit message: cleaned up

File: champ_description/urdf/accessories.urdf.xacro (robot description, xacro)
@@ -21,7 +21,4 @@
         <origin xyz="${base_x_length / 2} 0.0 ${base_z_length / 2 + 0.01}" rpy="0 0 0"/>
     </xacro:sensor_xtion>
-    <gazebo reference="hokuyo_frame">
-		<material>Gazebo/FlatBlack</material>
-	</gazebo>
     <gazebo>
         <plugin name="imu_controller" filename="libhector_gazebo_ros_imu.so">

Commit message: changed sensor plugin from local to hector_sensors_description

File: champ_description/urdf/accessories.urdf.xacro (robot description, xacro)
@@ -1,7 +1,7 @@
 <?xml version="1.0"?>
 <robot xmlns:xacro="http://ros.org/wiki/xacro">
-    <xacro:include filename="$(find common_sensors)/urdf/sensors/hokuyo_utm30lx.urdf.xacro" />
-    <xacro:include filename="$(find common_sensors)/urdf/sensors/xtion.urdf.xacro" />
-    <!-- <xacro:hokuyo_utm30lx
+    <xacro:include filename="$(find hector_sensors_description)/urdf/hokuyo_utm30lx.urdf.xacro" />
+    <xacro:include filename="$(find hector_sensors_description)/urdf/asus_camera.urdf.xacro" />
+    <xacro:hokuyo_utm30lx
         name="hokuyo"
         parent="base_link"
@@ -15,10 +15,10 @@
     <gazebo reference="hokuyo_frame">
 		<material>Gazebo/FlatBlack</material>
-	</gazebo> -->
-    <xacro:sensor_xtion
+	</gazebo>
+    <xacro:asus_camera_model
         parent="base_link"
-        camera_name="camera">
+        name="camera">
         <origin xyz="${base_x_length / 2} 0.0 ${base_z_length / 2 + 0.01}" rpy="0 0 0"/>
-    </xacro:sensor_xtion>
+    </xacro:asus_camera_model>
     <gazebo>
         <plugin name="imu_controller" filename="libhector_gazebo_ros_imu.so">

File: champ_description/urdf/champ.urdf (robot description, URDF)
Before this commit: robot champ, 28 links, 27 joints
Links:
- removed link camera_base_frame
- removed link camera_depth_frame
- removed link camera_depth_optical_frame
- removed link camera_link
- removed link camera_rgb_frame
- removed link camera_rgb_optical_frame
- removed link imu_link
Joints:
- removed joint camera_base_joint
- removed joint camera_depth_joint
- removed joint camera_depth_optical_joint
- removed joint camera_joint
- removed joint camera_rgb_joint
- removed joint camera_rgb_optical_joint
- removed joint imu_joint

File: champ_description/urdf/champ.urdf.xacro (robot description, xacro)
@@ -26,8 +26,4 @@
         </visual>
     </link>
-    <!-- <joint name="base_champ_joint" type="fixed">
-        <parent link="champ" />
-        <child link="base_link" />
-    </joint> -->
     <gazebo reference="base_link">
         <material>Gazebo/FlatBlack</material>

Commit message: added manipulator

File: champ_description/urdf/accessories.urdf.xacro (robot description, xacro)
@@ -46,3 +46,7 @@
         <child link="imu_link" />
     </joint>
+    <!-- <xacro:include filename="$(find champ_arm_description)/urdf/champ_arm.urdf.xacro" />
+    <xacro:champ_arm parent="base_link">
+        <origin xyz="0.07 0.0 ${base_z_length / 2}" rpy="0 0 0"/>
+    </xacro:champ_arm> -->
 </robot>

Commit message: added velodyne

File: champ_description/urdf/accessories.urdf.xacro (robot description, xacro)
@@ -45,5 +45,9 @@
         <child link="imu_link" />
     </joint>
-    <!-- <xacro:include filename="$(find champ_arm_description)/urdf/champ_arm.urdf.xacro" />
+    <!-- <xacro:include filename="$(find velodyne_description)/urdf/VLP-16.urdf.xacro"/>
+    <xacro:VLP-16 parent="base_link" name="velodyne" topic="velodyne_points" hz="10" samples="1024" gpu="false" lasers="16" max_range="100">
+        <origin xyz="0 0 ${base_z_length / 2}" rpy="0 0 0" />
+    </xacro:VLP-16>
+    <xacro:include filename="$(find champ_arm_description)/urdf/champ_arm.urdf.xacro" />
     <xacro:champ_arm parent="base_link">
         <origin xyz="0.07 0.0 ${base_z_length / 2}" rpy="0 0 0"/>

Commit message: shifted the depth sensor below the

File: champ_description/urdf/accessories.urdf.xacro (robot description, xacro)
@@ -19,5 +19,5 @@
         parent="base_link"
         name="camera">
-        <origin xyz="${base_x_length / 2} 0.0 ${base_z_length / 2 + 0.01}" rpy="0 0 0"/>
+        <origin xyz="${base_x_length / 2} 0.0 -${base_z_length / 2 + 0.01}" rpy="0 0 0"/>
     </xacro:asus_camera>
     <gazebo>

File: champ_description/urdf/champ.urdf (robot description, URDF)
Before this commit: robot champ, 29 links, 28 joints
Joints:
- joint camera_joint: origin xyz=0.25 0.0 0.075 rpy=0 0 0 -> xyz=0.25 0.0 -0.075 rpy=0 0 0

Commit message: fixed spawning of multiple robots

File: champ_description/urdf/accessories.urdf.xacro (robot description, xacro)
@@ -1,55 +1,54 @@
 <?xml version="1.0"?>
 <robot xmlns:xacro="http://ros.org/wiki/xacro">
-    <xacro:include filename="$(find hector_sensors_description)/urdf/hokuyo_utm30lx.urdf.xacro" />
-    <xacro:include filename="$(find hector_sensors_description)/urdf/asus_camera.urdf.xacro" />
-    <xacro:hokuyo_utm30lx
-        name="hokuyo"
-        parent="base_link"
-        ros_topic="scan"
-        update_rate="30"
-        ray_count="1040"
-        min_angle="130"
-        max_angle="-130" >
-        <origin xyz="0.0 0.0 ${base_z_length / 2 + 0.04}" rpy="0 0 0"/>
-    </xacro:hokuyo_utm30lx>
-    <gazebo reference="hokuyo_frame">
-		<material>Gazebo/FlatBlack</material>
-	</gazebo>
-    <xacro:asus_camera
-        parent="base_link"
-        name="camera">
-        <origin xyz="${base_x_length / 2} 0.0 -${base_z_length / 2 + 0.01}" rpy="0 0 0"/>
-    </xacro:asus_camera>
-    <gazebo>
-        <plugin name="imu_controller" filename="libhector_gazebo_ros_imu.so">
-            <updateRate>50.0</updateRate>
-            <bodyName>imu_link</bodyName>
-            <topicName>imu/data</topicName>
-            <accelDrift>0.005 0.005 0.005</accelDrift>
-            <accelGaussianNoise>0.005 0.005 0.005</accelGaussianNoise>
-            <rateDrift>0.005 0.005 0.005 </rateDrift>
-            <rateGaussianNoise>0.005 0.005 0.005 </rateGaussianNoise>
-            <headingDrift>0.005</headingDrift>
-            <headingGaussianNoise>0.005</headingGaussianNoise>
-        </plugin>
-    </gazebo>
-    <link name="imu_link">
-        <inertial>
-            <mass value="0.001"/>
-            <origin xyz="0 0 0" rpy="0 0 0"/>
-            <inertia ixx="1e-09" ixy="0.0" ixz="0.0" iyy="1e-09" iyz="0.0" izz="1e-09"/>
-        </inertial>
-    </link>
-    <joint name="imu_joint" type="fixed">
-        <parent link="base_link" />
-        <child link="imu_link" />
-    </joint>
-    <!-- <xacro:include filename="$(find velodyne_description)/urdf/VLP-16.urdf.xacro"/>
-    <xacro:VLP-16 parent="base_link" name="velodyne" topic="velodyne_points" hz="10" samples="1024" gpu="false" lasers="16" max_range="100">
-        <origin xyz="0 0 ${base_z_length / 2}" rpy="0 0 0" />
-    </xacro:VLP-16>
-    <xacro:include filename="$(find champ_arm_description)/urdf/champ_arm.urdf.xacro" />
-    <xacro:champ_arm parent="base_link">
-        <origin xyz="0.07 0.0 ${base_z_length / 2}" rpy="0 0 0"/>
-    </xacro:champ_arm> -->
+    <xacro:macro name="accessories" params="base_name base_length base_height  " >
+        <xacro:include filename="$(find hector_sensors_description)/urdf/hokuyo_utm30lx.urdf.xacro" />
+        <xacro:include filename="$(find hector_sensors_description)/urdf/asus_camera.urdf.xacro" />
+        <xacro:hokuyo_utm30lx
+            name="hokuyo"
+            parent="${base_name}"
+            ros_topic="scan"
+            update_rate="30"
+            ray_count="1040"
+            min_angle="130"
+            max_angle="-130" >
+            <origin xyz="0.0 0.0 ${base_height / 2 + 0.04}" rpy="0 0 0"/>
+        </xacro:hokuyo_utm30lx>
+        <xacro:asus_camera
+            parent="${base_name}"
+            name="camera">
+            <origin xyz="${base_length / 2} 0.0 -${base_height / 2 + 0.01}" rpy="0 0 0"/>
+        </xacro:asus_camera>
+        <gazebo>
+            <plugin name="imu_controller" filename="libhector_gazebo_ros_imu.so">
+                <updateRate>50.0</updateRate>
+                <bodyName>imu_link</bodyName>
+                <topicName>imu/data</topicName>
+                <accelDrift>0.005 0.005 0.005</accelDrift>
+                <accelGaussianNoise>0.005 0.005 0.005</accelGaussianNoise>
+                <rateDrift>0.005 0.005 0.005 </rateDrift>
+                <rateGaussianNoise>0.005 0.005 0.005 </rateGaussianNoise>
+                <headingDrift>0.005</headingDrift>
+                <headingGaussianNoise>0.005</headingGaussianNoise>
+            </plugin>
+        </gazebo>
+        <link name="imu_link">
+            <inertial>
+                <mass value="0.001"/>
+                <origin xyz="0 0 0" rpy="0 0 0"/>
+                <inertia ixx="1e-09" ixy="0.0" ixz="0.0" iyy="1e-09" iyz="0.0" izz="1e-09"/>
+            </inertial>
+        </link>
+        <joint name="imu_joint" type="fixed">
+            <parent link="${base_name}" />
+            <child link="imu_link" />
+        </joint>
+        <!-- <xacro:include filename="$(find velodyne_description)/urdf/VLP-16.urdf.xacro"/>
+        <xacro:VLP-16 parent="${base_name}" name="velodyne" topic="velodyne_points" hz="10" samples="1024" gpu="false" lasers="16" max_range="100">
+            <origin xyz="0 0 ${base_height / 2}" rpy="0 0 0" />
+        </xacro:VLP-16>
+        <xacro:include filename="$(find champ_arm_description)/urdf/champ_arm.urdf.xacro" />
+        <xacro:champ_arm parent="${base_name}">
+            <origin xyz="0.07 0.0 ${base_height / 2}" rpy="0 0 0"/>
+        </xacro:champ_arm> -->
+    </xacro:macro>
 </robot>

File: champ_description/urdf/champ.urdf.xacro (robot description, xacro)
@@ -37,4 +37,9 @@
     <xacro:include filename="$(find champ_description)/urdf/leg.urdf.xacro" />
     <xacro:include filename="$(find champ_description)/urdf/accessories.urdf.xacro" />
+    <xacro:accessories
+        base_name="base_link"
+        base_length="${base_x_length}"
+        base_height="${base_z_length}"
+    />
     <xacro:champ_leg leg="lf"/>
     <xacro:champ_leg leg="lh"/>

Commit message: Port description and gazebo, urdf is working, but ros2_control is not yet

File: champ_description/urdf/accessories.urdf.xacro (robot description, xacro)
@@ -2,6 +2,6 @@
 <robot xmlns:xacro="http://ros.org/wiki/xacro">
     <xacro:macro name="accessories" params="base_name base_length base_height  " >
-        <xacro:include filename="$(find hector_sensors_description)/urdf/hokuyo_utm30lx.urdf.xacro" />
-        <xacro:include filename="$(find hector_sensors_description)/urdf/asus_camera.urdf.xacro" />
+        <xacro:include filename="$(find champ_description)/urdf/hokuyo_utm30lx.urdf.xacro" />
+        <xacro:include filename="$(find champ_description)/urdf/asus_camera.urdf.xacro" />
         <xacro:hokuyo_utm30lx
             name="hokuyo"
@@ -19,17 +19,4 @@
             <origin xyz="${base_length / 2} 0.0 -${base_height / 2 + 0.01}" rpy="0 0 0"/>
         </xacro:asus_camera>
-        <gazebo>
-            <plugin name="imu_controller" filename="libhector_gazebo_ros_imu.so">
-                <updateRate>50.0</updateRate>
-                <bodyName>imu_link</bodyName>
-                <topicName>imu/data</topicName>
-                <accelDrift>0.005 0.005 0.005</accelDrift>
-                <accelGaussianNoise>0.005 0.005 0.005</accelGaussianNoise>
-                <rateDrift>0.005 0.005 0.005 </rateDrift>
-                <rateGaussianNoise>0.005 0.005 0.005 </rateGaussianNoise>
-                <headingDrift>0.005</headingDrift>
-                <headingGaussianNoise>0.005</headingGaussianNoise>
-            </plugin>
-        </gazebo>
         <link name="imu_link">
             <inertial>
@@ -38,4 +25,23 @@
                 <inertia ixx="1e-09" ixy="0.0" ixz="0.0" iyy="1e-09" iyz="0.0" izz="1e-09"/>
             </inertial>
+            <sensor name="imu_controller" type="imu">
+                <always_on>true</always_on>
+                <update_rate>50</update_rate>
+                <plugin name="gazebo_ros_imu_sensor" filename="libgazebo_ros_imu_sensor.so">
+                    <ros>
+                        <namespace>/imu</namespace>
+                        <argument>~/out:=data</argument>
+                    </ros>
+                    <!-- <updateRate>50.0</updateRate>
+                    <bodyName>imu_link</bodyName>
+                    <topicName>imu/data</topicName>
+                    <accelDrift>0.005 0.005 0.005</accelDrift>
+                    <accelGaussianNoise>0.005 0.005 0.005</accelGaussianNoise>
+                    <rateDrift>0.005 0.005 0.005 </rateDrift>
+                    <rateGaussianNoise>0.005 0.005 0.005 </rateGaussianNoise>
+                    <headingDrift>0.005</headingDrift>
+                    <headingGaussianNoise>0.005</headingGaussianNoise> -->
+                </plugin>
+            </sensor>
         </link>
         <joint name="imu_joint" type="fixed">

File: champ_description/urdf/champ.urdf (robot description, URDF)
Before this commit: robot champ, 29 links, 28 joints
Links:
- link base_link: geometry collision mesh filename=$(find champ_description)/meshes/base.stl scale=0.001 0.001 0.001; visual mesh filename=$(find champ_description)/meshes/base.stl scale=0.001 0.001 0.001
- link camera_link: geometry collision mesh filename=$(find champ_description)/meshes/asus_camera_simple.dae; visual mesh filename=$(find champ_description)/meshes/asus_camera_simple.dae
- link hokuyo_frame: geometry collision box size=0.058 0.058 0.087; visual mesh filename=$(find champ_description)/meshes/hokuyo_utm_30lx.dae

File: champ_description/urdf/champ.urdf.xacro (robot description, xacro)
@@ -13,5 +13,5 @@
             <origin xyz="0 0 0" rpy="0 0 0" />
             <geometry>
-                <mesh filename="package://champ_description/meshes/base.stl" scale="0.001 0.001 0.001" />
+                <mesh filename="file://$(find champ_description)/meshes/base.stl" scale="0.001 0.001 0.001" />
             </geometry>
             <material name="black" />
@@ -48,18 +48,27 @@
     <gazebo>
       <plugin name="p3d_base_controller" filename="libgazebo_ros_p3d.so">
-            <alwaysOn>true</alwaysOn>
-            <updateRate>10.0</updateRate>
-            <bodyName>base_link</bodyName>
-            <topicName>odom/ground_truth</topicName>
-            <gaussianNoise>0.01</gaussianNoise>
-            <frameName>world</frameName>
-            <xyzOffsets>0 0 0</xyzOffsets>
-            <rpyOffsets>0 0 0</rpyOffsets>
-        </plugin>
+            <ros>
+                <namespace>/demo</namespace>
+                <argument>odom:=odom/ground_truth</argument>
+            </ros>
+            <body_name>base_link</body_name>
+            <frame_name>world</frame_name>
+            <update_rate>10.0</update_rate>
+            <xyz_offset>0 0 0</xyz_offset>
+            <rpy_offset>0 0 0</rpy_offset>
+            <gaussian_noise>0.01</gaussian_noise>
+    </plugin>
     </gazebo>
-    <gazebo>
+    <!-- <gazebo>
         <plugin name="gazebo_ros_control" filename="libgazebo_ros_control.so">
             <legacyModeNS>true</legacyModeNS>
         </plugin>
+    </gazebo> -->
+    <gazebo>
+    <plugin filename="libgazebo_ros2_control.so" name="gazebo_ros2_control">
+        <robot_param>robot_description</robot_param>
+        <robot_param_node>robot_state_publisher</robot_param_node>
+        <parameters>$(find champ_gazebo)/config/ros_control.yaml</parameters>
+      </plugin>
     </gazebo>
 </robot>

File: champ_description/urdf/leg.urdf.xacro (robot description, xacro)
@@ -132,5 +132,5 @@
             <origin xyz="0 0 -${lower_leg_to_foot_distance}" rpy="0 0 0" />
         </joint>
-        <transmission name="${leg}_hip_joint_trans">
+        <!-- <transmission name="${leg}_hip_joint_trans">
             <type>transmission_interface/SimpleTransmission</type>
             <joint name="${leg}_hip_joint">
@@ -161,5 +161,5 @@
                 <mechanicalReduction>1</mechanicalReduction>
             </actuator>
-        </transmission>
+        </transmission> -->
     </xacro:macro>
 </robot>

File: champ_description/urdf/properties.urdf.xacro (robot description, xacro)
@@ -6,20 +6,20 @@
     <xacro:property name="upper_leg_to_lower_leg_distance" value="0.141" />
     <xacro:property name="lower_leg_to_foot_distance" value="0.141" />
-    <xacro:property name="hip_mesh_path" value="package://champ_description/meshes/hip.stl" />
+    <xacro:property name="hip_mesh_path" value="file://$(find champ_description)/meshes/hip.stl" />
     <xacro:property name="hip_mass" value="0.250" />
     <xacro:property name="hip_x_length" value="0.112" />
     <xacro:property name="hip_y_length" value="0.08" />
     <xacro:property name="hip_z_length" value="0.130" />
-    <xacro:property name="upper_leg_mesh_path" value="package://champ_description/meshes/upper_leg.stl" />
+    <xacro:property name="upper_leg_mesh_path" value="file://$(find champ_description)/meshes/upper_leg.stl" />
     <xacro:property name="upper_leg_mass" value="0.125" />
     <xacro:property name="upper_leg_x_length" value="0.05" />
     <xacro:property name="upper_leg_y_length" value="0.03" />
     <xacro:property name="upper_leg_z_length" value="0.1905" />
-    <xacro:property name="lower_leg_mesh_path" value="package://champ_description/meshes/lower_leg.stl" />
+    <xacro:property name="lower_leg_mesh_path" value="file://$(find champ_description)/meshes/lower_leg.stl" />
     <xacro:property name="lower_leg_mass" value="0.125" />
     <xacro:property name="lower_leg_x_length" value="0.039" />
     <xacro:property name="lower_leg_y_length" value="0.022" />
     <xacro:property name="lower_leg_z_length" value="0.156" />
-    <xacro:property name="base_mesh_path" value="package://champ_description/meshes/base.stl" />
+    <xacro:property name="base_mesh_path" value="file://$(find champ_description)/meshes/base.stl" />
     <xacro:property name="base_mass" value="2.0" />
     <xacro:property name="base_x_length" value="0.5" />
