Commit message: Fix wobble gait in gazebo

File: champ_description/urdf/accessories.urdf.xacro (robot description, xacro)
@@ -25,23 +25,4 @@
                 <inertia ixx="1e-09" ixy="0.0" ixz="0.0" iyy="1e-09" iyz="0.0" izz="1e-09"/>
             </inertial>
-            <sensor name="imu_controller" type="imu">
-                <always_on>true</always_on>
-                <update_rate>50</update_rate>
-                <plugin name="gazebo_ros_imu_sensor" filename="libgazebo_ros_imu_sensor.so">
-                    <ros>
-                        <namespace>/imu</namespace>
-                        <argument>~/out:=data</argument>
-                    </ros>
-                    <!-- <updateRate>50.0</updateRate>
-                    <bodyName>imu_link</bodyName>
-                    <topicName>imu/data</topicName>
-                    <accelDrift>0.005 0.005 0.005</accelDrift>
-                    <accelGaussianNoise>0.005 0.005 0.005</accelGaussianNoise>
-                    <rateDrift>0.005 0.005 0.005 </rateDrift>
-                    <rateGaussianNoise>0.005 0.005 0.005 </rateGaussianNoise>
-                    <headingDrift>0.005</headingDrift>
-                    <headingGaussianNoise>0.005</headingGaussianNoise> -->
-                </plugin>
-            </sensor>
         </link>
         <joint name="imu_joint" type="fixed">
@@ -49,4 +30,25 @@
             <child link="imu_link" />
         </joint>
+        <gazebo reference="imu_link">
+                <sensor name="imu_controller" type="imu">
+                    <always_on>true</always_on>
+                    <update_rate>50</update_rate>
+                    <plugin name="gazebo_ros_imu_sensor" filename="libgazebo_ros_imu_sensor.so">
+                        <ros>
+                            <namespace>/imu</namespace>
+                            <argument>~/out:=data</argument>
+                        </ros>
+                        <!-- <updateRate>50.0</updateRate>
+                        <bodyName>imu_link</bodyName>
+                        <topicName>imu/data</topicName>
+                        <accelDrift>0.005 0.005 0.005</accelDrift>
+                        <accelGaussianNoise>0.005 0.005 0.005</accelGaussianNoise>
+                        <rateDrift>0.005 0.005 0.005 </rateDrift>
+                        <rateGaussianNoise>0.005 0.005 0.005 </rateGaussianNoise>
+                        <headingDrift>0.005</headingDrift>
+                        <headingGaussianNoise>0.005</headingGaussianNoise> -->
+                    </plugin>
+                </sensor>
+            </gazebo>
         <!-- <xacro:include filename="$(find velodyne_description)/urdf/VLP-16.urdf.xacro"/>
         <xacro:VLP-16 parent="${base_name}" name="velodyne" topic="velodyne_points" hz="10" samples="1024" gpu="false" lasers="16" max_range="100">

File: champ_description/urdf/champ.urdf (robot description, URDF)
Before this commit: robot champ, 29 links, 28 joints
Links:
- link base_link: geometry collision mesh filename=file:///home/Alexander.Karavaev/champ_ws/install/champ_desc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 scale=0.001 0.001 0.001; visual mesh filename=file:///home/Alexander.Karavaev/champ_ws/install/champ_desc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 scale=0.001 0.001 0.001
- link camera_link: geometry collision mesh filename=file:///home/Alexander.Karavaev/champ_ws/install/champ_desc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; visual mesh filename=file:///home/Alexander.Karavaev/champ_ws/install/champ_desc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
- link hokuyo_frame: geometry collision box size=0.058 0.058 0.087; visual mesh filename=file:///home/Alexander.Karavaev/champ_ws/install/champ_desc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
- link lf_hip_link: geometry collision mesh filename=file:///home/Alexander.Karavaev/champ_ws/install/champ_desc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 scale=0.001 0.001 0.001; visual mesh filename=file:///home/Alexander.Karavaev/champ_ws/install/champ_desc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 scale=0.001 0.001 0.001
- link lf_lower_leg_link: geometry collision mesh filename=file:///home/Alexander.Karavaev/champ_ws/install/champ_desc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 scale=0.001 0.001 0.001; visual mesh filename=file:///home/Alexander.Karavaev/champ_ws/install/champ_desc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 scale=0.001 0.001 0.001
- link lf_upper_leg_link: geometry collision mesh filename=file:///home/Alexander.Karavaev/champ_ws/install/champ_desc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 scale=0.001 0.001 0.001; visual mesh filename=file:///home/Alexander.Karavaev/champ_ws/install/champ_desc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 scale=0.001 0.001 0.001
- link lh_hip_link: geometry collision mesh filename=file:///home/Alexander.Karavaev/champ_ws/install/champ_desc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 scale=0.001 0.001 0.001; visual mesh filename=file:///home/Alexander.Karavaev/champ_ws/install/champ_desc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 scale=0.001 0.001 0.001
- link lh_lower_leg_link: geometry collision mesh filename=file:///home/Alexander.Karavaev/champ_ws/install/champ_desc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 scale=0.001 0.001 0.001; visual mesh filename=file:///home/Alexander.Karavaev/champ_ws/install/champ_desc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 scale=0.001 0.001 0.001
- link lh_upper_leg_link: geometry collision mesh filename=file:///home/Alexander.Karavaev/champ_ws/install/champ_desc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 scale=0.001 0.001 0.001; visual mesh filename=file:///home/Alexander.Karavaev/champ_ws/install/champ_desc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 scale=0.001 0.001 0.001
- link rf_hip_link: geometry collision mesh filename=file:///home/Alexander.Karavaev/champ_ws/install/champ_desc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 scale=0.001 0.001 0.001; visual mesh filename=file:///home/Alexander.Karavaev/champ_ws/install/champ_desc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 scale=0.001 0.001 0.001
- link rf_lower_leg_link: geometry collision mesh filename=file:///home/Alexander.Karavaev/champ_ws/install/champ_desc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 scale=0.001 0.001 0.001; visual mesh filename=file:///home/Alexander.Karavaev/champ_ws/install/champ_desc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 scale=0.001 0.001 0.001
- link rf_upper_leg_link: geometry collision mesh filename=file:///home/Alexander.Karavaev/champ_ws/install/champ_desc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 scale=0.001 0.001 0.001; visual mesh filename=file:///home/Alexander.Karavaev/champ_ws/install/champ_desc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 scale=0.001 0.001 0.001
- link rh_hip_link: geometry collision mesh filename=file:///home/Alexander.Karavaev/champ_ws/install/champ_desc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 scale=0.001 0.001 0.001; visual mesh filename=file:///home/Alexander.Karavaev/champ_ws/install/champ_desc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 scale=0.001 0.001 0.001
- link rh_lower_leg_link: geometry collision mesh filename=file:///home/Alexander.Karavaev/champ_ws/install/champ_desc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 scale=0.001 0.001 0.001; visual mesh filename=file:///home/Alexander.Karavaev/champ_ws/install/champ_desc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 scale=0.001 0.001 0.001
- link rh_upper_leg_link: geometry collision mesh filename=file:///home/Alexander.Karavaev/champ_ws/install/champ_desc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 scale=0.001 0.001 0.001; visual mesh filename=file:///home/Alexander.Karavaev/champ_ws/install/champ_desc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 scale=0.001 0.001 0.001
Joints:
- joint camera_depth_optical_joint: origin xyz=0 0 0 rpy=-1.57079632679 0.0 -1.57079632679 -> xyz=0 0 0 rpy=-1.5707963267948966 0.0 -1.5707963267948966
- joint camera_rgb_optical_joint: origin xyz=0 0 0 rpy=-1.57079632679 0.0 -1.57079632679 -> xyz=0 0 0 rpy=-1.5707963267948966 0.0 -1.5707963267948966
- joint hokuyo_joint: origin xyz=0.0 0.0 0.105 rpy=0 0 0 -> xyz=0.0 0.0 0.10500000000000001 rpy=0 0 0
- joint lf_foot_joint: origin xyz=0 0 -0.141 rpy=0 0 0 -> xyz=0.00325 0 -0.141 rpy=0 0 0
- joint lf_hip_joint: limit lower=-3.14159265359 upper=3.14159265359 effort=25 velocity=1.5 -> lower=-3.141592653589793 upper=3.141592653589793 effort=25 velocity=1.5
- joint lf_lower_leg_joint: limit lower=-3.14159265359 upper=3.14159265359 effort=25 velocity=1.5 -> lower=-3.141592653589793 upper=3.141592653589793 effort=25 velocity=1.5
- joint lf_upper_leg_joint: limit lower=-3.14159265359 upper=3.14159265359 effort=25 velocity=1.5 -> lower=-3.141592653589793 upper=3.141592653589793 effort=25 velocity=1.5
- joint lh_foot_joint: origin xyz=0 0 -0.141 rpy=0 0 0 -> xyz=0.00325 0 -0.141 rpy=0 0 0
- joint lh_hip_joint: limit lower=-3.14159265359 upper=3.14159265359 effort=25 velocity=1.5 -> lower=-3.141592653589793 upper=3.141592653589793 effort=25 velocity=1.5
- joint lh_lower_leg_joint: limit lower=-3.14159265359 upper=3.14159265359 effort=25 velocity=1.5 -> lower=-3.141592653589793 upper=3.141592653589793 effort=25 velocity=1.5
- joint lh_upper_leg_joint: limit lower=-3.14159265359 upper=3.14159265359 effort=25 velocity=1.5 -> lower=-3.141592653589793 upper=3.141592653589793 effort=25 velocity=1.5
- joint rf_foot_joint: origin xyz=0 0 -0.141 rpy=0 0 0 -> xyz=0.00325 0 -0.141 rpy=0 0 0
- joint rf_hip_joint: limit lower=-3.14159265359 upper=3.14159265359 effort=25 velocity=1.5 -> lower=-3.141592653589793 upper=3.141592653589793 effort=25 velocity=1.5
- joint rf_lower_leg_joint: limit lower=-3.14159265359 upper=3.14159265359 effort=25 velocity=1.5 -> lower=-3.141592653589793 upper=3.141592653589793 effort=25 velocity=1.5
- joint rf_upper_leg_joint: limit lower=-3.14159265359 upper=3.14159265359 effort=25 velocity=1.5 -> lower=-3.141592653589793 upper=3.141592653589793 effort=25 velocity=1.5
- joint rh_foot_joint: origin xyz=0 0 -0.141 rpy=0 0 0 -> xyz=0.00325 0 -0.141 rpy=0 0 0
- joint rh_hip_joint: limit lower=-3.14159265359 upper=3.14159265359 effort=25 velocity=1.5 -> lower=-3.141592653589793 upper=3.141592653589793 effort=25 velocity=1.5
- joint rh_lower_leg_joint: limit lower=-3.14159265359 upper=3.14159265359 effort=25 velocity=1.5 -> lower=-3.141592653589793 upper=3.141592653589793 effort=25 velocity=1.5
- joint rh_upper_leg_joint: limit lower=-3.14159265359 upper=3.14159265359 effort=25 velocity=1.5 -> lower=-3.141592653589793 upper=3.141592653589793 effort=25 velocity=1.5

File: champ_description/urdf/leg.urdf.xacro (robot description, xacro)
@@ -91,10 +91,9 @@
         </link>
         <gazebo reference="${leg}_lower_leg_link">
-            <kp>10000000.0</kp>
+            <kp>10000000000.0</kp>
             <kd>100.0</kd>
             <mu1>0.8</mu1>
             <mu2>0.8</mu2>
-            <maxVel>0.0</maxVel>
-            <minDepth>0.001</minDepth>
+            <minDepth>0.05</minDepth>
             <material>Gazebo/FlatBlack</material>
         </gazebo>
